File: ESP32_5V/ESP32_5V.kicad_pcb (KiCad board)
At the start: 4 copper layers, 90 x 70 mm, 76 parts, among them J1 Barrel_Jack_MountingPin, J10 Conn_01x11, J11 Conn_01x11, J12 Conn_01x11, J13 Conn_01x11, J15 Screw_Terminal_01x11, J16 Screw_Terminal_01x11, J2 Conn_01x11, J3 Conn_01x11, J4 Conn_01x11, J5 Conn_01x11, J6 Conn_01x11, J7 Conn_01x11, J8 Conn_01x11, J9 Conn_01x11, U1 TPS563201, U2 TPS563201, U3 SN74LVC245APW, U4 SN74LVC245APW, U5 SN74LVC245APW

Commit message: update
Parts:
- removed D4: 1N5819WS, Diode_SMD:D_SOD-323
- added R11: 1k, Resistor_SMD:R_0402_1005Metric, F.Cu at (124.1, 59.8)
- added R12: 1k, Resistor_SMD:R_0402_1005Metric, F.Cu at (124.1, 57.4)
- added R13: 1k, Resistor_SMD:R_0402_1005Metric, F.Cu at (154.5, 52.4)
- added R14: 1k, Resistor_SMD:R_0402_1005Metric, F.Cu at (154.5, 59.9)
- added R15: 1k, Resistor_SMD:R_0402_1005Metric, F.Cu at (154.5, 62.5)
- added R16: 1k, Resistor_SMD:R_0402_1005Metric, F.Cu at (154.5, 65.2)
- added R17: 1k, Resistor_SMD:R_0402_1005Metric, F.Cu at (154.5, 67.5)
- added R18: 1k, Resistor_SMD:R_0402_1005Metric, F.Cu at (154.5, 70.2)
- added R19: 1k, Resistor_SMD:R_0402_1005Metric, F.Cu at (154.5, 72.7)
- added R20: 1k, Resistor_SMD:R_0402_1005Metric, F.Cu at (154.5, 75.1)
- added R21: 1k, Resistor_SMD:R_0402_1005Metric, F.Cu at (154.5, 77.8)
- added R22: 1k, Resistor_SMD:R_0402_1005Metric, F.Cu at (154.5, 80.2)
- added R23: 1k, Resistor_SMD:R_0402_1005Metric, F.Cu at (124.1, 80.2)
- added R24: 1k, Resistor_SMD:R_0402_1005Metric, F.Cu at (124.1, 77.8)
- added R25: 1k, Resistor_SMD:R_0402_1005Metric, F.Cu at (124.1, 75.0)
- added R26: 1k, Resistor_SMD:R_0402_1005Metric, F.Cu at (124.1, 72.5)
- added R27: 1k, Resistor_SMD:R_0402_1005Metric, F.Cu at (124.1, 70.0)
- added R28: 1k, Resistor_SMD:R_0402_1005Metric, F.Cu at (124.1, 67.6)
- added R29: 1k, Resistor_SMD:R_0402_1005Metric, F.Cu at (124.1, 65.0)
- added R30: 1k, Resistor_SMD:R_0402_1005Metric, F.Cu at (124.1, 62.5)
- C10, C11, C16, C17, C18, C19, C20, C21, C22, C23, C30, C31, C32, C8, C9: footprint Capacitor_SMD:C_0402_1005Metric -> Capacitor_SMD:C_1206_3216Metric
- C2, C3: footprint Capacitor_SMD:C_1210_3225Metric -> Capacitor_SMD:C_0402_1005Metric
- C25, C26, C29: value 100nF -> 10nF
- R10: value 500 -> 390
- R8: value 500 -> 100
- R9: value 500 -> 150
- moved R1 96.3 mm to (179.7, 104.8), turned to 90 degrees
- moved C23 32.0 mm to (172.9, 85.8)
- moved C19 31.9 mm to (161.7, 85.8)
- moved C16 31.9 mm to (114.8, 85.7)
- moved C20 31.9 mm to (104.2, 85.8)
- moved C4 14.5 mm to (140.8, 109.0), turned to 90 degrees
- moved C5 12.8 mm to (115.0, 108.2), turned to 90 degrees
- moved C2 12.6 mm to (143.2, 108.9), turned to 90 degrees
- moved C11 10.7 mm to (124.6, 101.8), turned to -90 degrees
- moved C3 9.80 mm to (117.3, 108.2), turned to 90 degrees
- moved C10 9.54 mm to (150.4, 102.6), turned to -90 degrees
- moved TP2 9.10 mm to (115.2, 96.5)
- moved R5 7.59 mm to (148.9, 110.3), turned to -90 degrees
- moved R7 7.39 mm to (123.5, 109.6), turned to -90 degrees
- moved L2 7.32 mm to (120.0, 101.8), turned to 90 degrees
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Connections:
- C30 pad 1: Net-(D4-K) -> +5V
- H1 pad 1: Net-(H1-Pad1) -> unconnected-(H1-Pad1)_8
- H3 pad 1: unconnected-(H3-Pad1) -> Net-(H3-Pad1)
- JP1 pad 2: Net-(D4-K) -> +5V
- R1 pad 1: Net-(H1-Pad1) -> Net-(H3-Pad1)
Routing:
- net GND: track 59.3 -> 101.0 mm, vias 78 -> 93
- net Net-(D4-K): track 6.22 -> 0.00 mm
- net Net-(H1-Pad1): track 4.16 -> 0.00 mm
- net /Conector_5V/D5_5V: track 63.3 -> 67.2 mm
- net /Conector_5V/D22_5V: track 74.6 -> 78.5 mm
- net /Conector_5V/D19_5V: track 68.9 -> 72.8 mm
- net /Conector_5V/D35_5V: track 71.9 -> 75.7 mm
- net /Conector_5V/D13_5V: track 44.4 -> 48.1 mm
- net /Conector_5V/D14_5V: track 50.8 -> 54.1 mm
- net Net-(U2-VFB): track 6.26 -> 3.08 mm
- net Net-(U1-VFB): track 5.92 -> 2.81 mm
- net /Conector_5V/D26_5V: track 57.1 -> 60.1 mm
- net /Conector_5V/D15_5V: track 44.9 -> 47.7 mm
- net /Conector_5V/D4_5V: track 50.7 -> 53.5 mm
- net /Conector_5V/D33_5V: track 63.3 -> 65.8 mm
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- added copper zone on F.Cu, net +3V3

Commit message: update
Routing:
- net GND: track 101.0 -> 100.9 mm, vias 93 -> 92

Commit message: update
Parts:
- removed JP1: Jumper_2_Open, Connector_PinHeader_2.54mm:PinHeader_1x02_P2.54mm_Vertical
- added D4: 1N5712UR, Diode_SMD:D_MELF, F.Cu at (120.8, 87.3)
- moved D2 3.55 mm to (108.3, 110.6)
- moved R10 3.55 mm to (109.5, 108.5)
- moved D1 3.55 mm to (107.2, 110.6)
- moved D3 3.55 mm to (109.5, 110.6)
- moved R8 3.55 mm to (107.2, 108.5)
- moved R9 3.55 mm to (108.3, 108.5)
- moved R29 1.19 mm to (122.9, 65.0)
- moved R27 1.19 mm to (122.9, 70.0)
- moved R28 1.19 mm to (122.9, 67.6)
- moved R30 1.14 mm to (123.0, 62.4)
- moved R12 1.14 mm to (123.0, 57.4)
- moved R11 1.14 mm to (123.0, 59.8)
- moved R23 1.14 mm to (123.0, 80.2)
- moved R26 1.14 mm to (123.0, 72.5)
- moved R24 1.10 mm to (123.0, 77.8)
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Connections:
- C30 pad 1: +5V -> Net-(D4-K)
- J14 pad 15: Net-(JP1-A) -> Net-(D4-K)
Routing:
- net Net-(D4-K): track 0.00 -> 7.88 mm
- net Net-(JP1-A): track 6.12 -> 0.00 mm
- net GND: track 100.9 -> 102.2 mm, vias 92 -> 110
- net /Conector_3V3/D33: track 45.5 -> 46.7 mm
- net /Conector_3V3/D26: track 39.9 -> 41.1 mm
- net /Conector_3V3/D25: track 42.7 -> 43.9 mm
- net /Conector_3V3/D32: track 48.3 -> 49.5 mm
- net /Conector_3V3/D34: track 55.2 -> 56.4 mm
- net /Conector_3V3/D27: track 37.1 -> 38.2 mm
- net /Conector_3V3/D13: track 28.6 -> 29.8 mm
- net /Conector_3V3/D35: track 52.5 -> 53.6 mm
- net /Conector_3V3/D14: track 34.3 -> 35.4 mm
- net /Conector_3V3/D12: track 31.6 -> 32.7 mm
- net /Conector_3V3/D19: track 48.5 -> 49.3 mm
- net /Conector_3V3/D5: track 42.9 -> 43.7 mm
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