File: ESP32_5V/Conector_3V3.kicad_sch (KiCad schematic)
At the start: 6 parts, among them J12 Conn_01x11, J13 Conn_01x11, J14 Conn_01x11, J7 Conn_01x11, J8 Conn_01x11, J9 Conn_01x11

Commit message: update
Parts:
- renumbered J8 to J2, J12 to J3, J13 to J4, J9 to J5, J7 to J6, J14 to J7
Other:
- moved on the sheet: J2, J3, J4, J5, J6, J7

Commit message: update
Connections:
- net D23 is gone; now on net D19: J7.3 (Pin_3)
- net D12: no longer J7.1 (Pin_1)
- net D13: no longer J7.2 (Pin_2)
- net D15: now also J7.10 (Pin_10)
- net D16: now also J7.7 (Pin_7); no longer J7.10 (Pin_10)
- net D17: now also J7.6 (Pin_6); no longer J7.9 (Pin_9)
- net D18: now also J7.4 (Pin_4); no longer J7.7 (Pin_7)
- net D19: no longer J7.6 (Pin_6)
- net D2: now also J7.9 (Pin_9)
- net D21: now also J7.2 (Pin_2); no longer J7.5 (Pin_5)
- net D22: now also J7.1 (Pin_1); no longer J7.4 (Pin_4)
- net D4: now also J7.8 (Pin_8); no longer J7.11 (Pin_11)
- net D5: now also J7.5 (Pin_5); no longer J7.8 (Pin_8)
- no-connect marks 0 -> 2
Other:
- note added: "Conector derecho 3V3"
- note added: "Conector izquierdo 3V3"
- moved on the sheet: J2, J3, J4, J5, J6

Commit message: update
Parts:
- added C14, C15, C16, C17: 10u, Capacitor_SMD:C_0402_1005Metric, symbol Device:C
Connections:
- net +3V3: now also C14.1, C15.1, C16.1, C17.1
- net GND: now also C14.2, C15.2, C16.2, C17.2

Commit message: update
Parts:
- renumbered C14 to C16, C15 to C17, C16 to C18, C17 to C19
Changed lines of the file:
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@@
 		(dnp no)
 		(fields_autoplaced yes)
-		(property "Reference" "#PWR04"
+		(property "Reference" "#PWR027"
 			(at 57.15 68.58 0)
 			(effects
@@
 			(project ""
 				(path "/a7bda8b3-4b40-4c73-a9d2-e587ed8710cd/d42efb0d-e007-4d41-bee2-3d89ed4ea0d8"
-					(reference "#PWR04")
+					(reference "#PWR027")
 					(unit 1)
 				)
@@
 		(dnp no)
 		(fields_autoplaced yes)
-		(property "Reference" "#PWR038"
+		(property "Reference" "#PWR029"
 			(at 92.71 53.34 0)
 			(effects
@@
 			(project "ESP32_5V"
 				(path "/a7bda8b3-4b40-4c73-a9d2-e587ed8710cd/d42efb0d-e007-4d41-bee2-3d89ed4ea0d8"
-					(reference "#PWR038")
+					(reference "#PWR029")
 					(unit 1)
 				)
@@
 		(on_board yes)
 		(dnp no)
-		(property "Reference" "C14"
+		(property "Reference" "C16"
 			(at 80.772 36.83 0)
 			(effects
@@
 			(project "ESP32_5V"
 				(path "/a7bda8b3-4b40-4c73-a9d2-e587ed8710cd/d42efb0d-e007-4d41-bee2-3d89ed4ea0d8"
-					(reference "C14")
+					(reference "C16")
 					(unit 1)
 				)
@@
 		(dnp no)
 		(fields_autoplaced yes)
-		(property "Reference" "#PWR05"
+		(property "Reference" "#PWR030"
 			(at 113.03 133.35 0)
 			(effects
@@
 			(project ""
 				(path "/a7bda8b3-4b40-4c73-a9d2-e587ed8710cd/d42efb0d-e007-4d41-bee2-3d89ed4ea0d8"
-					(reference "#PWR05")
+					(reference "#PWR030")
 					(unit 1)
 				)
@@
 		(on_board yes)
 		(dnp no)
-		(property "Reference" "C17"
+		(property "Reference" "C19"
 			(at 111.252 36.83 0)
 			(effects
@@
 			(project "ESP32_5V"
 				(path "/a7bda8b3-4b40-4c73-a9d2-e587ed8710cd/d42efb0d-e007-4d41-bee2-3d89ed4ea0d8"
-					(reference "C17")
+					(reference "C19")
 					(unit 1)
 				)
@@
 		(on_board yes)
 		(dnp no)
-		(property "Reference" "C16"
+		(property "Reference" "C18"
 			(at 101.092 36.83 0)
 			(effects
@@
 			(project "ESP32_5V"
 				(path "/a7bda8b3-4b40-4c73-a9d2-e587ed8710cd/d42efb0d-e007-4d41-bee2-3d89ed4ea0d8"
-					(reference "C16")
+					(reference "C18")
 					(unit 1)
 				)
@@
 		(on_board yes)
 		(dnp no)
-		(property "Reference" "C15"
+		(property "Reference" "C17"
 			(at 90.932 36.83 0)
 			(effects
@@
 			(project "ESP32_5V"
 				(path "/a7bda8b3-4b40-4c73-a9d2-e587ed8710cd/d42efb0d-e007-4d41-bee2-3d89ed4ea0d8"
-					(reference "C15")
+					(reference "C17")
 					(unit 1)
 				)
@@
 		(dnp no)
 		(fields_autoplaced yes)
-		(property "Reference" "#PWR040"
+		(property "Reference" "#PWR028"
 			(at 92.71 34.29 0)
 			(effects
@@
 			(project "ESP32_5V"
 				(path "/a7bda8b3-4b40-4c73-a9d2-e587ed8710cd/d42efb0d-e007-4d41-bee2-3d89ed4ea0d8"
-					(reference "#PWR040")
-					(unit 1)
-				)
+					(reference "#PWR028")
+					(unit 1)
+				)

Commit message: update
Parts:
- C16, C17, C18, C19: footprint Capacitor_SMD:C_0402_1005Metric -> Capacitor_SMD:C_1206_3216Metric
Changed lines of the file:
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@@
 			)
 		)
-		(property "Footprint" "Capacitor_SMD:C_0402_1005Metric"
+		(property "Footprint" "Capacitor_SMD:C_1206_3216Metric"
 			(at 78.4352 41.91 0)
 			(effects
@@
 			)
 		)
-		(property "Footprint" "Capacitor_SMD:C_0402_1005Metric"
+		(property "Footprint" "Capacitor_SMD:C_1206_3216Metric"
 			(at 108.9152 41.91 0)
 			(effects
@@
 			)
 		)
-		(property "Footprint" "Capacitor_SMD:C_0402_1005Metric"
+		(property "Footprint" "Capacitor_SMD:C_1206_3216Metric"
 			(at 98.7552 41.91 0)
 			(effects
@@
 			)
 		)
-		(property "Footprint" "Capacitor_SMD:C_0402_1005Metric"
+		(property "Footprint" "Capacitor_SMD:C_1206_3216Metric"
 			(at 88.5952 41.91 0)
 			(effects
