File: ESP32_5V/conector_atornillado.kicad_sch (KiCad schematic)
At the start: 2 parts, among them J5 Screw_Terminal_01x11, J6 Screw_Terminal_01x11

Commit message: update
Parts:
- renumbered J5 to J15, J6 to J16
Other:
- moved on the sheet: J15, J16

Commit message: update
Parts:
- J15, J16: symbol Connector:Screw_Terminal_01x11 -> Connector:Screw_Terminal_01x12
Connections:
- net D23_5V is gone; now on net +5V: J15.11 (Pin_11)
- net +5V: now reaches J16.11 (Pin_11)
- new net GND: J15.12 (Pin_12), J16.12 (Pin_12)
- no-connect marks 1 -> 0
Other:
- note added: "Conectores atronillados"

Commit message: update
Parts:
- added C25, C27: 10u, Capacitor_SMD:C_0402_1005Metric, symbol Device:C
Connections:
- net +5V: now also C25.1, C27.1
- net GND: now also C25.2, C27.2

Commit message: update
Parts:
- renumbered C27 to C31, C25 to C32

Commit message: update
Parts:
- C31, C32: footprint Capacitor_SMD:C_0402_1005Metric -> Capacitor_SMD:C_1206_3216Metric
Changed lines of the file:
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@@
 			)
 		)
-		(property "Footprint" "Capacitor_SMD:C_0402_1005Metric"
+		(property "Footprint" "Capacitor_SMD:C_1206_3216Metric"
 			(at 195.2752 143.51 0)
 			(effects
@@
 			)
 		)
-		(property "Footprint" "Capacitor_SMD:C_0402_1005Metric"
+		(property "Footprint" "Capacitor_SMD:C_1206_3216Metric"
 			(at 112.7252 143.51 0)
 			(effects
