File: ESP32_5V/Alimentaciones.kicad_sch (KiCad schematic)
At the start: 1 part, among them J17 Jack-DC

Commit message: update
Parts:
- added D1: LED, symbol Device:LED
- added R7: 10k, symbol Device:R_US
- added TP1: TestPoint, symbol Connector:TestPoint
- J1: renamed from J17; footprint (none) -> Connector_BarrelJack:BarrelJack_GCT_DCJ200-10-A_Horizontal
Connections:
- net +5V: now also R7.1, TP1.1
- net GND: now also D1.1 (K)
- new net: D1.2 (A), R7.2

Commit message: update
Parts:
- removed J1: Jack-DC, Connector_BarrelJack:BarrelJack_GCT_DCJ200-10-A_Horizontal, symbol Connector:Jack-DC
- added C10, C9: 10u, Capacitor_SMD:C_0402_1005Metric, symbol Device:C
- added C7: 10u, Capacitor_SMD:C_1210_3225Metric, symbol Device:C
- added C8: 100nF, Capacitor_SMD:C_0402_1005Metric, symbol Device:C
- added D2: LED, LED_SMD:LED_0402_1005Metric, symbol Device:LED
- added J17: Barrel_Jack_MountingPin, Connector_BarrelJack:BarrelJack_GCT_DCJ200-10-A_Horizontal, symbol Connector:Barrel_Jack_MountingPin
- added L1: 4,7uH, Inductor_SMD:L_6.3x6.3_H3, symbol Device:L
- added R10: 20k, Resistor_SMD:R_0402_1005Metric, symbol Device:R_US
- added R4, R8: 10k, Resistor_SMD:R_0402_1005Metric, symbol Device:R_US
- added R9: 110k, Resistor_SMD:R_0402_1005Metric, symbol Device:R_US
- added TP2: TestPoint, TestPoint:TestPoint_Pad_D2.0mm, symbol Connector:TestPoint
- added U4: TPS563201, Package_TO_SOT_SMD:SOT-23-6, symbol drones_devices:TPS563201
- D1: footprint (none) -> LED_SMD:LED_0402_1005Metric
- R7: footprint (none) -> Resistor_SMD:R_0402_1005Metric
- TP1: footprint (none) -> TestPoint:TestPoint_Pad_D2.0mm
Connections:
- net +5V: now also C10.1, C9.1, L1.2, R9.1
- net GND: now also C10.2, C7.2, C9.2, D2.1 (K), J17.2, J17.MP (MountPin), R10.2, U4.1 (GND)
- net VCC: now also C7.1, J17.1, R4.1, R8.2, TP2.1, U4.3 (IN)
- new net: R8.1, U4.5 (EN)
- new net: R10.1, R9.2, U4.4 (VFB)
- new net: C8.1, U4.6 (VBST)
- new net: C8.2, L1.1, U4.2 (SW)
- new net: D2.2 (A), R4.2
Other:
- note added: "Conversor de Vcc a +5V"

Commit message: update
Parts:
- added C11, C6: 10u, Capacitor_SMD:C_0402_1005Metric, symbol Device:C
- added C4: 100n, Capacitor_SMD:C_1210_3225Metric, symbol Device:C
- added C5: 10u, Capacitor_SMD:C_1210_3225Metric, symbol Device:C
- R4, R7: value 10k -> 500
Connections:
- net +5V: now also C11.1, C6.1
- net GND: now also C11.2, C4.2, C5.2, C6.2
- net VCC: now also C4.1, C5.1

Commit message: update
Parts:
- removed C6: 10u, Capacitor_SMD:C_0402_1005Metric, symbol Device:C
- added C3: 100n, Capacitor_SMD:C_1210_3225Metric, symbol Device:C
- added C5: 10u, Capacitor_SMD:C_1210_3225Metric, symbol Device:C
- added C7: 100nF, Capacitor_SMD:C_0402_1005Metric, symbol Device:C
- added C9: 10u, Capacitor_SMD:C_0402_1005Metric, symbol Device:C
- added D1: LED, LED_SMD:LED_0402_1005Metric, symbol Device:LED
- added L2: 4,7uH, Inductor_SMD:L_6.3x6.3_H3, symbol Device:L
- added R3, R7: 10k, Resistor_SMD:R_0402_1005Metric, symbol Device:R_US
- added R6: 33k, Resistor_SMD:R_0402_1005Metric, symbol Device:R_US
- added R8: 500, Resistor_SMD:R_0402_1005Metric, symbol Device:R_US
- added TP2: TestPoint, TestPoint:TestPoint_Pad_D2.0mm, symbol Connector:TestPoint
- added U2: TPS563201, Package_TO_SOT_SMD:SOT-23-6, symbol drones_devices:TPS563201
- R4: renamed from R9; value 110k -> 51k
- R5: renamed from R10; value 20k -> 10k
- renumbered C5 to C1, C4 to C2, C7 to C4, C8 to C6, C9 to C8, D1 to D2, D2 to D3, J17 to J1, R4 to R10, R8 to R2, R7 to R9, TP2 to TP1, TP1 to TP3, U4 to U1
Connections:
- net +5V: no longer C11.1
- net GND: now also C3.2, C5.2, C9.2, D1.1 (K), R7.2, U2.1 (GND)
- net VCC: now also C3.1, C5.1, R3.2, U2.3 (IN)
- new net: R3.1, U2.5 (EN)
- new net: D1.2 (A), R8.2
- new net: R6.2, R7.1, U2.4 (VFB)
- new net: C7.1, U2.6 (VBST)
- new net: C7.2, L2.1, U2.2 (SW)
- new net +3V3: C11.1, C9.1, L2.2, R6.1, R8.1, TP2.1

Commit message: update
Parts:
- C10, C11, C8, C9: footprint Capacitor_SMD:C_0402_1005Metric -> Capacitor_SMD:C_1206_3216Metric
- C2, C3: footprint Capacitor_SMD:C_1210_3225Metric -> Capacitor_SMD:C_0402_1005Metric
- R10: value 500 -> 390
- R8: value 500 -> 100
- R9: value 500 -> 150
Changed lines of the file:
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@@
 			)
 		)
-		(property "Footprint" "Capacitor_SMD:C_0402_1005Metric"
+		(property "Footprint" "Capacitor_SMD:C_1206_3216Metric"
 			(at 141.9352 96.52 0)
 			(effects
@@
 			)
 		)
-		(property "Value" "500"
+		(property "Value" "100"
 			(at 213.36 71.1199 0)
 			(effects
@@
 			)
 		)
-		(property "Footprint" "Capacitor_SMD:C_0402_1005Metric"
+		(property "Footprint" "Capacitor_SMD:C_1206_3216Metric"
 			(at 147.0152 144.78 0)
 			(effects
@@
 			)
 		)
-		(property "Value" "500"
+		(property "Value" "150"
 			(at 223.52 71.1199 0)
 			(effects
@@
 			)
 		)
-		(property "Footprint" "Capacitor_SMD:C_1210_3225Metric"
+		(property "Footprint" "Capacitor_SMD:C_0402_1005Metric"
 			(at 69.5452 97.79 0)
 			(effects
@@
 			)
 		)
-		(property "Footprint" "Capacitor_SMD:C_0402_1005Metric"
+		(property "Footprint" "Capacitor_SMD:C_1206_3216Metric"
 			(at 152.0952 96.52 0)
 			(effects
@@
 			)
 		)
-		(property "Footprint" "Capacitor_SMD:C_0402_1005Metric"
+		(property "Footprint" "Capacitor_SMD:C_1206_3216Metric"
 			(at 157.1752 144.78 0)
 			(effects
@@
 			)
 		)
-		(property "Value" "500"
+		(property "Value" "390"
 			(at 236.22 71.1199 0)
 			(effects
@@
 			)
 		)
-		(property "Footprint" "Capacitor_SMD:C_1210_3225Metric"
+		(property "Footprint" "Capacitor_SMD:C_0402_1005Metric"
 			(at 74.6252 146.05 0)
 			(effects

Commit message: update
Parts:
- C2, C3, C6, C7: footprint Capacitor_SMD:C_0402_1005Metric -> Capacitor_SMD:C_0805_2012Metric_Pad1.18x1.45mm_HandSolder
- D1, D2, D3: footprint LED_SMD:LED_0402_1005Metric -> LED_SMD:LED_0805_2012Metric_Pad1.15x1.40mm_HandSolder
- R10, R2, R3, R4, R5, R6, R7, R8, R9: footprint Resistor_SMD:R_0402_1005Metric -> Resistor_SMD:R_0805_2012Metric_Pad1.20x1.40mm_HandSolder
Changed lines of the file:
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@@
 			)
 		)
-		(property "Footprint" "Resistor_SMD:R_0402_1005Metric"
+		(property "Footprint" "Resistor_SMD:R_0805_2012Metric_Pad1.20x1.40mm_HandSolder"
 			(at 211.836 70.104 90)
 			(hide yes)
@@
 			)
 		)
-		(property "Footprint" "Resistor_SMD:R_0402_1005Metric"
+		(property "Footprint" "Resistor_SMD:R_0805_2012Metric_Pad1.20x1.40mm_HandSolder"
 			(at 97.536 143.256 90)
 			(hide yes)
@@
 			)
 		)
-		(property "Footprint" "Resistor_SMD:R_0402_1005Metric"
+		(property "Footprint" "Resistor_SMD:R_0805_2012Metric_Pad1.20x1.40mm_HandSolder"
 			(at 92.456 94.996 90)
 			(hide yes)
@@
 			)
 		)
-		(property "Footprint" "Resistor_SMD:R_0402_1005Metric"
+		(property "Footprint" "Resistor_SMD:R_0805_2012Metric_Pad1.20x1.40mm_HandSolder"
 			(at 135.636 141.224 90)
 			(hide yes)
@@
 			)
 		)
-		(property "Footprint" "LED_SMD:LED_0402_1005Metric"
+		(property "Footprint" "LED_SMD:LED_0805_2012Metric_Pad1.15x1.40mm_HandSolder"
 			(at 210.82 80.01 0)
 			(hide yes)
@@
 			)
 		)
-		(property "Footprint" "Resistor_SMD:R_0402_1005Metric"
+		(property "Footprint" "Resistor_SMD:R_0805_2012Metric_Pad1.20x1.40mm_HandSolder"
 			(at 130.556 100.584 90)
 			(hide yes)
@@
 			)
 		)
-		(property "Footprint" "Capacitor_SMD:C_0402_1005Metric"
+		(property "Footprint" "Capacitor_SMD:C_0805_2012Metric_Pad1.18x1.45mm_HandSolder"
 			(at 116.84 76.5048 0)
 			(hide yes)
@@
 			)
 		)
-		(property "Footprint" "Capacitor_SMD:C_0402_1005Metric"
+		(property "Footprint" "Capacitor_SMD:C_0805_2012Metric_Pad1.18x1.45mm_HandSolder"
 			(at 121.92 124.7648 0)
 			(hide yes)
@@
 			)
 		)
-		(property "Footprint" "Resistor_SMD:R_0402_1005Metric"
+		(property "Footprint" "Resistor_SMD:R_0805_2012Metric_Pad1.20x1.40mm_HandSolder"
 			(at 221.996 70.104 90)
 			(hide yes)
@@
 			)
 		)
-		(property "Footprint" "Capacitor_SMD:C_0402_1005Metric"
+		(property "Footprint" "Capacitor_SMD:C_0805_2012Metric_Pad1.18x1.45mm_HandSolder"
 			(at 69.5452 97.79 0)
 			(hide yes)
@@
 			)
 		)
-		(property "Footprint" "Resistor_SMD:R_0402_1005Metric"
+		(property "Footprint" "Resistor_SMD:R_0805_2012Metric_Pad1.20x1.40mm_HandSolder"
 			(at 130.556 92.964 90)
 			(hide yes)
@@
 			)
 		)
-		(property "Footprint" "LED_SMD:LED_0402_1005Metric"
+		(property "Footprint" "LED_SMD:LED_0805_2012Metric_Pad1.15x1.40mm_HandSolder"
 			(at 233.68 80.01 0)
 			(hide yes)
@@
 			)
 		)
-		(property "Footprint" "LED_SMD:LED_0402_1005Metric"
+		(property "Footprint" "LED_SMD:LED_0805_2012Metric_Pad1.15x1.40mm_HandSolder"
 			(at 220.98 80.01 0)
 			(hide yes)
@@
 			)
 		)
-		(property "Footprint" "Resistor_SMD:R_0402_1005Metric"
+		(property "Footprint" "Resistor_SMD:R_0805_2012Metric_Pad1.20x1.40mm_HandSolder"
 			(at 234.696 70.104 90)
 			(hide yes)
@@
 			)
 		)
-		(property "Footprint" "Capacitor_SMD:C_0402_1005Metric"
+		(property "Footprint" "Capacitor_SMD:C_0805_2012Metric_Pad1.18x1.45mm_HandSolder"
 			(at 74.6252 146.05 0)
 			(hide yes)
@@
 			)
 		)
-		(property "Footprint" "Resistor_SMD:R_0402_1005Metric"
+		(property "Footprint" "Resistor_SMD:R_0805_2012Metric_Pad1.20x1.40mm_HandSolder"
 			(at 135.636 148.844 90)
 			(hide yes)
