File: ESP32_5V/Conector_5V.kicad_sch (KiCad schematic)
At the start: 21 parts, among them J1 Conn_01x11, J10 Conn_01x11, J11 Conn_01x11, J15 Conn_01x11, J16 Conn_01x11, J4 Conn_01x11, U1 TXS0108EPW, U2 TXS0108EPW, U3 TXS0108EPW

Commit message: update
Parts:
- C1: renamed from C3; now not fitted
- C2, C5: now not fitted
- renumbered C4 to C3, C1 to C4, J15 to J12, J16 to J13, J1 to J8, J4 to J9, R3 to R2, R2 to R3
Changed lines of the file:
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@@
 		(dnp no)
 		(fields_autoplaced yes)
-		(property "Reference" "#PWR013"
+		(property "Reference" "#PWR017"
 			(at 144.78 116.84 0)
 			(effects
@@
 			(project "ESP32_5V"
 				(path "/a7bda8b3-4b40-4c73-a9d2-e587ed8710cd/c7c1796f-3147-43e6-887b-773c57671428"
-					(reference "#PWR013")
+					(reference "#PWR017")
 					(unit 1)
 				)
@@
 		(dnp no)
 		(fields_autoplaced yes)
-		(property "Reference" "#PWR010"
+		(property "Reference" "#PWR012"
 			(at 139.7 43.18 0)
 			(effects
@@
 			(project ""
 				(path "/a7bda8b3-4b40-4c73-a9d2-e587ed8710cd/c7c1796f-3147-43e6-887b-773c57671428"
-					(reference "#PWR010")
+					(reference "#PWR012")
 					(unit 1)
 				)
@@
 		(in_bom yes)
 		(on_board yes)
-		(dnp no)
-		(property "Reference" "C3"
+		(dnp yes)
+		(property "Reference" "C1"
 			(at 135.128 38.354 90)
 			(effects
@@
 			(project "ESP32_5V"
 				(path "/a7bda8b3-4b40-4c73-a9d2-e587ed8710cd/c7c1796f-3147-43e6-887b-773c57671428"
-					(reference "C3")
+					(reference "C1")
 					(unit 1)
 				)
@@
 		(dnp no)
 		(fields_autoplaced yes)
-		(property "Reference" "#PWR015"
+		(property "Reference" "#PWR020"
 			(at 172.72 96.52 0)
 			(effects
@@
 			(project "ESP32_5V"
 				(path "/a7bda8b3-4b40-4c73-a9d2-e587ed8710cd/c7c1796f-3147-43e6-887b-773c57671428"
-					(reference "#PWR015")
+					(reference "#PWR020")
 					(unit 1)
 				)
@@
 		(dnp no)
 		(fields_autoplaced yes)
-		(property "Reference" "#PWR027"
+		(property "Reference" "#PWR025"
 			(at 219.71 85.09 0)
 			(effects
@@
 			(project "ESP32_5V"
 				(path "/a7bda8b3-4b40-4c73-a9d2-e587ed8710cd/c7c1796f-3147-43e6-887b-773c57671428"
-					(reference "#PWR027")
+					(reference "#PWR025")
 					(unit 1)
 				)
@@
 		(dnp no)
 		(fields_autoplaced yes)
-		(property "Reference" "#PWR019"
+		(property "Reference" "#PWR07"
 			(at 52.07 173.99 0)
 			(effects
@@
 			(project ""
 				(path "/a7bda8b3-4b40-4c73-a9d2-e587ed8710cd/c7c1796f-3147-43e6-887b-773c57671428"
-					(reference "#PWR019")
+					(reference "#PWR07")
 					(unit 1)
 				)
@@
 		(dnp no)
 		(fields_autoplaced yes)
-		(property "Reference" "#PWR017"
+		(property "Reference" "#PWR023"
 			(at 204.47 134.62 0)
 			(effects
@@
 			(project "ESP32_5V"
 				(path "/a7bda8b3-4b40-4c73-a9d2-e587ed8710cd/c7c1796f-3147-43e6-887b-773c57671428"
-					(reference "#PWR017")
+					(reference "#PWR023")
 					(unit 1)
 				)
@@
 		(in_bom yes)
 		(on_board yes)
-		(dnp no)
+		(dnp yes)
 		(property "Reference" "C2"
 			(at 135.128 112.014 90)
@@
 		(dnp no)
 		(fields_autoplaced yes)
-		(property "Reference" "#PWR016"
+		(property "Reference" "#PWR022"
 			(at 201.93 78.74 0)
 			(effects
@@
 			(project "ESP32_5V"
 				(path "/a7bda8b3-4b40-4c73-a9d2-e587ed8710cd/c7c1796f-3147-43e6-887b-773c57671428"
-					(reference "#PWR016")
+					(reference "#PWR022")
 					(unit 1)
 				)
@@
 		(dnp no)
 		(fields_autoplaced yes)
-		(property "Reference" "#PWR014"
+		(property "Reference" "#PWR015"
 			(at 142.24 173.99 0)
 			(effects
@@
 			(project "ESP32_5V"
 				(path "/a7bda8b3-4b40-4c73-a9d2-e587ed8710cd/c7c1796f-3147-43e6-887b-773c57671428"
-					(reference "#PWR014")
+					(reference "#PWR015")
 					(unit 1)
 				)
@@
 		(dnp no)
 		(fields_autoplaced yes)
-		(property "Reference" "#PWR024"
+		(property "Reference" "#PWR010"
 			(at 127 49.53 0)
 			(effects
@@
 			(project "ESP32_5V"
 				(path "/a7bda8b3-4b40-4c73-a9d2-e587ed8710cd/c7c1796f-3147-43e6-887b-773c57671428"
-					(reference "#PWR024")
+					(reference "#PWR010")
 					(unit 1)
 				)
@@
 		(on_board yes)
 		(dnp no)
-		(property "Reference" "C4"
+		(property "Reference" "C3"
 			(at 149.352 38.354 90)
 			(effects
@@
 			(project "ESP32_5V"
 				(path "/a7bda8b3-4b40-4c73-a9d2-e587ed8710cd/c7c1796f-3147-43e6-887b-773c57671428"
-					(reference "C4")
+					(reference "C3")
 					(unit 1)
 				)
@@
 		(dnp no)
 		(fields_autoplaced yes)
-		(property "Reference" "#PWR026"
+		(property "Reference" "#PWR021"
 			(at 189.23 85.09 0)
 			(effects
@@
 			(project "ESP32_5V"
 				(path "/a7bda8b3-4b40-4c73-a9d2-e587ed8710cd/c7c1796f-3147-43e6-887b-773c57671428"
-					(reference "#PWR026")
+					(reference "#PWR021")
 					(unit 1)
 				)
@@
 		(dnp no)
 		(fields_autoplaced yes)
-		(property "Reference" "J15"
+		(property "Reference" "J12"
 			(at 262.89 55.8799 0)
 			(effects
@@
 			(project "ESP32_5V"
 				(path "/a7bda8b3-4b40-4c73-a9d2-e587ed8710cd/c7c1796f-3147-43e6-887b-773c57671428"
-					(reference "J15")
+					(reference "J12")
 					(unit 1)
 				)
@@
 		(dnp no)
 		(fields_autoplaced yes)
-		(property "Reference" "#PWR011"
+		(property "Reference" "#PWR09"
 			(at 110.49 134.62 0)
 			(effects
@@
 			(project "ESP32_5V"
 				(path "/a7bda8b3-4b40-4c73-a9d2-e587ed8710cd/c7c1796f-3147-43e6-887b-773c57671428"
-					(reference "#PWR011")
+					(reference "#PWR09")
 					(unit 1)
 				)
@@
 		(dnp no)
 		(fields_autoplaced yes)
-		(property "Reference" "#PWR08"
+		(property "Reference" "#PWR016"
 			(at 144.78 43.18 0)
 			(effects
@@
 			(project ""
 				(path "/a7bda8b3-4b40-4c73-a9d2-e587ed8710cd/c7c1796f-3147-43e6-887b-773c57671428"
-					(reference "#PWR08")
+					(reference "#PWR016")
 					(unit 1)
 				)
@@
 		(dnp no)
 		(fields_autoplaced yes)
-		(property "Reference" "#PWR04"
+		(property "Reference" "#PWR06"
 			(at 52.07 38.1 0)
 			(effects
@@
 			(project ""
 				(path "/a7bda8b3-4b40-4c73-a9d2-e587ed8710cd/c7c1796f-3147-43e6-887b-773c57671428"
-					(reference "#PWR04")
+					(reference "#PWR06")
 					(unit 1)
 				)
@@
 		(dnp no)
 		(fields_autoplaced yes)
-		(property "Reference" "J1"
+		(property "Reference" "J8"
 			(at 64.77 49.5299 0)
 			(effects
@@
 			(project ""
 				(path "/a7bda8b3-4b40-4c73-a9d2-e587ed8710cd/c7c1796f-3147-43e6-887b-773c57671428"
-					(reference "J1")
+					(reference "J8")
 					(unit 1)
 				)
@@
 		(dnp no)
 		(fields_autoplaced yes)
-		(property "Reference" "#PWR023"
+		(property "Reference" "#PWR011"
 			(at 127 123.19 0)
 			(effects
@@
 			(project "ESP32_5V"
 				(path "/a7bda8b3-4b40-4c73-a9d2-e587ed8710cd/c7c1796f-3147-43e6-887b-773c57671428"
-					(reference "#PWR023")
+					(reference "#PWR011")
 					(unit 1)
 				)
@@
 		(on_board yes)
 		(dnp no)
-		(property "Reference" "C1"
+		(property "Reference" "C4"
 			(at 149.352 112.014 90)
 			(effects
@@
 			(project ""
 				(path "/a7bda8b3-4b40-4c73-a9d2-e587ed8710cd/c7c1796f-3147-43e6-887b-773c57671428"
-					(reference "C1")
+					(reference "C4")
 					(unit 1)
 				)
@@
 		(on_board yes)
 		(dnp no)
-		(property "Reference" "R3"
+		(property "Reference" "R2"
 			(at 120.904 132.08 90)
 			(effects
@@
 			(project "ESP32_5V"
 				(path "/a7bda8b3-4b40-4c73-a9d2-e587ed8710cd/c7c1796f-3147-43e6-887b-773c57671428"
-					(reference "R3")
+					(reference "R2")
 					(unit 1)
 				)
@@
 		(dnp no)
 		(fields_autoplaced yes)
-		(property "Reference" "#PWR09"
+		(property "Reference" "#PWR014"
 			(at 142.24 99.06 0)
 			(effects
@@
 			(project "ESP32_5V"
 				(path "/a7bda8b3-4b40-4c73-a9d2-e587ed8710cd/c7c1796f-3147-43e6-887b-773c57671428"
-					(reference "#PWR09")
+					(reference "#PWR014")
 					(unit 1)
 				)
@@
 		(in_bom yes)
 		(on_board yes)
-		(dnp no)
+		(dnp yes)
 		(property "Reference" "C5"
 			(at 197.358 73.914 90)
@@
 		(dnp no)
 		(fields_autoplaced yes)
-		(property "Reference" "#PWR025"
+		(property "Reference" "#PWR018"
 			(at 157.48 49.53 0)
 			(effects
@@
 			(project "ESP32_5V"
 				(path "/a7bda8b3-4b40-4c73-a9d2-e587ed8710cd/c7c1796f-3147-43e6-887b-773c57671428"
-					(reference "#PWR025")
+					(reference "#PWR018")
 					(unit 1)
 				)
@@
 		(dnp no)
 		(fields_autoplaced yes)
-		(property "Reference" "#PWR018"
+		(property "Reference" "#PWR024"
 			(at 207.01 78.74 0)
 			(effects
@@
 			(project "ESP32_5V"
 				(path "/a7bda8b3-4b40-4c73-a9d2-e587ed8710cd/c7c1796f-3147-43e6-887b-773c57671428"
-					(reference "#PWR018")
+					(reference "#PWR024")
 					(unit 1)
 				)
@@
 		(dnp no)
 		(fields_autoplaced yes)
-		(property "Reference" "#PWR012"
+		(property "Reference" "#PWR013"
 			(at 139.7 116.84 0)
 			(effects
@@
 			(project "ESP32_5V"
 				(path "/a7bda8b3-4b40-4c73-a9d2-e587ed8710cd/c7c1796f-3147-43e6-887b-773c57671428"
-					(reference "#PWR012")
+					(reference "#PWR013")
 					(unit 1)
 				)
@@
 		(on_board yes)
 		(dnp yes)
-		(property "Reference" "R2"
+		(property "Reference" "R3"
 			(at 137.16 49.276 0)
 			(effects
@@
 			(project "ESP32_5V"
 				(path "/a7bda8b3-4b40-4c73-a9d2-e587ed8710cd/c7c1796f-3147-43e6-887b-773c57671428"
-					(reference "R2")
+					(reference "R3")
 					(unit 1)
 				)
@@
 		(dnp no)
 		(fields_autoplaced yes)
-		(property "Reference" "J4"
+		(property "Reference" "J9"
 			(at 64.77 80.0099 0)
 			(effects
@@
 			(project "ESP32_5V"
 				(path "/a7bda8b3-4b40-4c73-a9d2-e587ed8710cd/c7c1796f-3147-43e6-887b-773c57671428"
-					(reference "J4")
+					(reference "J9")
 					(unit 1)
 				)
@@
 		(dnp no)
 		(fields_autoplaced yes)
-		(property "Reference" "#PWR022"
+		(property "Reference" "#PWR019"
 			(at 157.48 123.19 0)
 			(effects
@@
 			(project "ESP32_5V"
 				(path "/a7bda8b3-4b40-4c73-a9d2-e587ed8710cd/c7c1796f-3147-43e6-887b-773c57671428"
-					(reference "#PWR022")
+					(reference "#PWR019")
 					(unit 1)
 				)
@@
 		(dnp no)
 		(fields_autoplaced yes)
-		(property "Reference" "J16"
+		(property "Reference" "J13"
 			(at 262.89 87.6299 0)
 			(effects
@@
 			(project "ESP32_5V"
 				(path "/a7bda8b3-4b40-4c73-a9d2-e587ed8710cd/c7c1796f-3147-43e6-887b-773c57671428"
-					(reference "J16")
+					(reference "J13")
 					(unit 1)
 				)
@@
 		(dnp no)
 		(fields_autoplaced yes)
-		(property "Reference" "#PWR07"
+		(property "Reference" "#PWR08"
 			(at 110.49 60.96 0)
 			(effects
@@
 			(project ""
 				(path "/a7bda8b3-4b40-4c73-a9d2-e587ed8710cd/c7c1796f-3147-43e6-887b-773c57671428"
-					(reference "#PWR07")
-					(unit 1)
-				)
+					(reference "#PWR08")
+					(unit 1)
+				)

Commit message: update
Parts:
- removed C4, C5, C6: 10nF, Capacitor_SMD:C_0402_1005Metric, symbol Device:C_Small
- removed R4, R6: 0, Resistor_SMD:R_0402_1005Metric, symbol Device:R_US
- removed R5: 10k, Resistor_SMD:R_0402_1005Metric, symbol Device:R_US
- removed U1, U2, U3: TXS0108EPW, Package_SO:TSSOP-20_4.4x6.5mm_P0.65mm, symbol Logic_LevelTranslator:TXS0108EPW
- added U1, U2, U5: SN74LVC245APW, Package_SO:TSSOP-20_4.4x6.5mm_P0.65mm, symbol Logic_LevelTranslator:SN74LVC245APW
- C1, C2, R3: now fitted
- R1, R2: value 10k -> 0
Connections:
- net +3V3 is gone; now on net +5V: C1.1, C2.1, R3.2
- net +5V: now also R1.2, R2.2, U1.20 (VCC), U2.20 (VCC), U5.20 (VCC)
- net D12: now also U1.2 (A1)
- net D12_5V: now also U1.18 (B1)
- net D13: now also U1.3 (A2)
- net D13_5V: now also U1.17 (B2)
- net D14: now also U5.9 (A8)
- net D14_5V: now also U5.11 (B8)
- net D15: now also U2.6 (A5)
- net D15_5V: now also U2.14 (B5)
- net D16: now also U2.3 (A2)
- net D16_5V: now also U2.17 (B2)
- net D17: now also U2.2 (A1)
- net D17_5V: now also U2.18 (B1)
- net D18: now also U1.8 (A7)
- net D18_5V: now also U1.12 (B7)
- net D19: now also U1.7 (A6)
- net D19_5V: now also U1.13 (B6)
- net D2: now also U2.5 (A4)
- net D21: now also U1.6 (A5)
- net D21_5V: now also U1.14 (B5)
- net D22: now also U1.5 (A4)
- net D22_5V: now also U1.15 (B4)
- net D25: now also U5.6 (A5)
- net D25_5V: now also U5.14 (B5)
- net D26: now also U5.7 (A6)
- net D26_5V: now also U5.13 (B6)
- net D27: now also U5.8 (A7)
- net D27_5V: now also U5.12 (B7)
- net D2_5V: now also U2.15 (B4)
- net D32: now also U5.4 (A3)
- net D32_5V: now also U5.16 (B3)
- net D33: now also U5.5 (A4)
- net D33_5V: now also U5.15 (B4)
- net D34: now also U5.2 (A1)
- net D34_5V: now also U5.18 (B1)
- net D35: now also U5.3 (A2)
- net D35_5V: now also U5.17 (B2)
- net D4: now also U2.4 (A3)
- net D4_5V: now also U2.16 (B3)
- net D5: now also U1.9 (A8)
- net D5_5V: now also U1.11 (B8)
- net GND: now also U1.10 (GND), U1.19 (~{OE}), U2.10 (GND), U2.19 (~{OE}), U5.10 (GND), U5.19 (~{OE}); no longer R1.1, R2.1
- net at R3.1: now also U2.1 (DIR); no longer R1.2
- net D23_5V: no longer names the net of J12.11 (Pin_11)
- new net: R1.1, U5.1 (DIR)
- new net: R2.1, U1.1 (DIR)
- no-connect marks 7 -> 10
Other:
- note added: "Conector derecho 5V"
- note added: "Conector izquierdo 5V"
- note added: "Drivers"
- moved on the sheet: C3, J10, J11, J13, J8, J9

Commit message: update
Parts:
- removed R1, R2, R3: 0, Resistor_SMD:R_0402_1005Metric, symbol Device:R_US
- added C18, C19, C20, C21: 10u, Capacitor_SMD:C_0402_1005Metric, symbol Device:C
- added C22, C23, C24: 100nF, Capacitor_SMD:C_0402_1005Metric, symbol Device:C_Small
- added RN1, RN2, RN3: R_Network08_US, Resistor_THT:R_Array_SIP9, symbol Device:R_Network08_US
- C1, C2, C3: value 10nF -> 100nF
Connections:
- net +5V: now also U1.1 (DIR), U2.1 (DIR), U5.1 (DIR), C18.1, C19.1, C20.1, C21.1, C22.1, C23.1, C24.1
- net D12: now also RN1.3 (R2)
- net D13: now also RN1.4 (R3)
- net D14: now also RN3.9 (R8)
- net D15: now also RN2.9 (R8)
- net D16: now also RN2.6 (R5)
- net D17: now also RN2.5 (R4)
- net D18: now also RN1.8 (R7)
- net D19: now also RN1.7 (R6)
- net D2: now also RN2.8 (R7)
- net D21: now also RN1.6 (R5)
- net D22: now also RN1.5 (R4)
- net D25: now also RN3.6 (R5)
- net D26: now also RN3.7 (R6)
- net D27: now also RN3.8 (R7)
- net D32: now also RN3.4 (R3)
- net D33: now also RN3.5 (R4)
- net D34: now also RN3.2 (R1)
- net D35: now also RN3.3 (R2)
- net D4: now also RN2.7 (R6)
- net D5: now also RN1.9 (R8)
- net GND: now also C18.2, C19.2, C20.2, C21.2, C22.2, C23.2, C24.2, RN1.1 (common), RN2.1 (common), RN3.1 (common)
- no-connect marks 10 -> 14

Commit message: update
Parts:
- removed RN1, RN2, RN3: R_Network08_US, Resistor_THT:R_Array_SIP9, symbol Device:R_Network08_US
- renumbered C18 to C20, C19 to C21, C20 to C22, C21 to C23, C22 to C24, C1 to C25, C24 to C26, C3 to C27, C23 to C28, C2 to C29, U1 to U3, U5 to U4, U2 to U5
Connections:
- net D12: now also U4.8 (A7); no longer U3.2 (A1)
- net D12_5V: now also U4.12 (B7); no longer U3.18 (B1)
- net D13: now also U4.9 (A8); no longer U3.3 (A2)
- net D13_5V: now also U4.11 (B8); no longer U3.17 (B2)
- net D14: now also U4.7 (A6); no longer U4.9 (A8)
- net D14_5V: now also U4.13 (B6); no longer U4.11 (B8)
- net D16: now also U5.9 (A8); no longer U5.3 (A2)
- net D16_5V: now also U5.11 (B8); no longer U5.17 (B2)
- net D17: now also U3.2 (A1); no longer U5.2 (A1)
- net D17_5V: now also U3.18 (B1); no longer U5.18 (B1)
- net D18: now also U3.4 (A3); no longer U3.8 (A7)
- net D18_5V: now also U3.16 (B3); no longer U3.12 (B7)
- net D19: now also U3.5 (A4); no longer U3.7 (A6)
- net D19_5V: now also U3.15 (B4); no longer U3.13 (B6)
- net D2: now also U5.7 (A6); no longer U5.5 (A4)
- net D22: now also U3.7 (A6); no longer U3.5 (A4)
- net D22_5V: now also U3.13 (B6); no longer U3.15 (B4)
- net D25: now also U4.4 (A3); no longer U4.6 (A5)
- net D25_5V: now also U4.16 (B3); no longer U4.14 (B5)
- net D26: now also U4.5 (A4); no longer U4.7 (A6)
- net D26_5V: now also U4.15 (B4); no longer U4.13 (B6)
- net D27: now also U4.6 (A5); no longer U4.8 (A7)
- net D27_5V: now also U4.14 (B5); no longer U4.12 (B7)
- net D2_5V: now also U5.13 (B6); no longer U5.15 (B4)
- net D32: now also U4.2 (A1); no longer U4.4 (A3)
- net D32_5V: now also U4.18 (B1); no longer U4.16 (B3)
- net D33: now also U4.3 (A2); no longer U4.5 (A4)
- net D33_5V: now also U4.17 (B2); no longer U4.15 (B4)
- net D34: now also U3.8 (A7); no longer U4.2 (A1)
- net D34_5V: now also U3.12 (B7); no longer U4.18 (B1)
- net D35: now also U3.9 (A8); no longer U4.3 (A2)
- net D35_5V: now also U3.11 (B8); no longer U4.17 (B2)
- net D4: now also U5.8 (A7); no longer U5.4 (A3)
- net D4_5V: now also U5.12 (B7); no longer U5.16 (B3)
- net D5: now also U3.3 (A2); no longer U3.9 (A8)
- net D5_5V: now also U3.17 (B2); no longer U3.11 (B8)
- no-connect marks 14 -> 6

Commit message: update
Parts:
- added R11, R12, R13, R14, R15, R16, R17, R18, R19, R20, R21, R22, R23, R24, R25, R26, R27, R28, R29, R30: 1k, Resistor_SMD:R_0402_1005Metric, symbol Device:R_US
- C20, C21, C22, C23: footprint Capacitor_SMD:C_0402_1005Metric -> Capacitor_SMD:C_1206_3216Metric
- C25, C26, C29: value 100nF -> 10nF
Connections:
- net D12: now also R24.1
- net D13: now also R23.1
- net D14: now also R25.1
- net D15: now also R22.1
- net D16: now also R19.1
- net D17: now also R18.1
- net D18: now also R16.1
- net D19: now also R15.1
- net D2: now also R21.1
- net D21: now also R14.1
- net D22: now also R13.1
- net D25: now also R28.1
- net D26: now also R27.1
- net D27: now also R26.1
- net D32: now also R30.1
- net D33: now also R29.1
- net D34: now also R12.1
- net D35: now also R11.1
- net D4: now also R20.1
- net D5: now also R17.1
- net GND: now also R11.2, R12.2, R13.2, R14.2, R15.2, R16.2, R17.2, R18.2, R19.2, R20.2, R21.2, R22.2, R23.2, R24.2, R25.2, R26.2, R27.2, R28.2, R29.2, R30.2
- no-connect marks 6 -> 10

Commit message: update
Parts:
- C24, C25, C26, C27, C28, C29: footprint Capacitor_SMD:C_0402_1005Metric -> Capacitor_SMD:C_0805_2012Metric_Pad1.18x1.45mm_HandSolder
- R11, R12, R13, R14, R15, R16, R17, R18, R19, R20, R21, R22, R23, R24, R25, R26, R27, R28, R29, R30: footprint Resistor_SMD:R_0402_1005Metric -> Resistor_SMD:R_0805_2012Metric_Pad1.20x1.40mm_HandSolder
Changed lines of the file:
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@@
 			)
 		)
-		(property "Footprint" "Resistor_SMD:R_0402_1005Metric"
+		(property "Footprint" "Resistor_SMD:R_0805_2012Metric_Pad1.20x1.40mm_HandSolder"
 			(at 256.286 148.844 90)
 			(hide yes)
@@
 			)
 		)
-		(property "Footprint" "Resistor_SMD:R_0402_1005Metric"
+		(property "Footprint" "Resistor_SMD:R_0805_2012Metric_Pad1.20x1.40mm_HandSolder"
 			(at 229.616 148.844 90)
 			(hide yes)
@@
 			)
 		)
-		(property "Footprint" "Capacitor_SMD:C_0402_1005Metric"
+		(property "Footprint" "Capacitor_SMD:C_0805_2012Metric_Pad1.18x1.45mm_HandSolder"
 			(at 118.11 107.95 0)
 			(hide yes)
@@
 			)
 		)
-		(property "Footprint" "Resistor_SMD:R_0402_1005Metric"
+		(property "Footprint" "Resistor_SMD:R_0805_2012Metric_Pad1.20x1.40mm_HandSolder"
 			(at 248.666 148.844 90)
 			(hide yes)
@@
 			)
 		)
-		(property "Footprint" "Resistor_SMD:R_0402_1005Metric"
+		(property "Footprint" "Resistor_SMD:R_0805_2012Metric_Pad1.20x1.40mm_HandSolder"
 			(at 271.526 148.844 90)
 			(hide yes)
@@
 			)
 		)
-		(property "Footprint" "Resistor_SMD:R_0402_1005Metric"
+		(property "Footprint" "Resistor_SMD:R_0805_2012Metric_Pad1.20x1.40mm_HandSolder"
 			(at 241.046 148.844 90)
 			(hide yes)
@@
 			)
 		)
-		(property "Footprint" "Resistor_SMD:R_0402_1005Metric"
+		(property "Footprint" "Resistor_SMD:R_0805_2012Metric_Pad1.20x1.40mm_HandSolder"
 			(at 218.186 148.844 90)
 			(hide yes)
@@
 			)
 		)
-		(property "Footprint" "Capacitor_SMD:C_0402_1005Metric"
+		(property "Footprint" "Capacitor_SMD:C_0805_2012Metric_Pad1.18x1.45mm_HandSolder"
 			(at 193.04 77.47 0)
 			(hide yes)
@@
 			)
 		)
-		(property "Footprint" "Resistor_SMD:R_0402_1005Metric"
+		(property "Footprint" "Resistor_SMD:R_0805_2012Metric_Pad1.20x1.40mm_HandSolder"
 			(at 221.996 148.844 90)
 			(hide yes)
@@
 			)
 		)
-		(property "Footprint" "Capacitor_SMD:C_0402_1005Metric"
+		(property "Footprint" "Capacitor_SMD:C_0805_2012Metric_Pad1.18x1.45mm_HandSolder"
 			(at 193.04 83.82 0)
 			(hide yes)
@@
 			)
 		)
-		(property "Footprint" "Resistor_SMD:R_0402_1005Metric"
+		(property "Footprint" "Resistor_SMD:R_0805_2012Metric_Pad1.20x1.40mm_HandSolder"
 			(at 210.566 148.844 90)
 			(hide yes)
@@
 			)
 		)
-		(property "Footprint" "Resistor_SMD:R_0402_1005Metric"
+		(property "Footprint" "Resistor_SMD:R_0805_2012Metric_Pad1.20x1.40mm_HandSolder"
 			(at 199.136 148.844 90)
 			(hide yes)
@@
 			)
 		)
-		(property "Footprint" "Resistor_SMD:R_0402_1005Metric"
+		(property "Footprint" "Resistor_SMD:R_0805_2012Metric_Pad1.20x1.40mm_HandSolder"
 			(at 233.426 148.844 90)
 			(hide yes)
@@
 			)
 		)
-		(property "Footprint" "Resistor_SMD:R_0402_1005Metric"
+		(property "Footprint" "Resistor_SMD:R_0805_2012Metric_Pad1.20x1.40mm_HandSolder"
 			(at 206.756 148.844 90)
 			(hide yes)
@@
 			)
 		)
-		(property "Footprint" "Resistor_SMD:R_0402_1005Metric"
+		(property "Footprint" "Resistor_SMD:R_0805_2012Metric_Pad1.20x1.40mm_HandSolder"
 			(at 260.096 148.844 90)
 			(hide yes)
@@
 			)
 		)
-		(property "Footprint" "Resistor_SMD:R_0402_1005Metric"
+		(property "Footprint" "Resistor_SMD:R_0805_2012Metric_Pad1.20x1.40mm_HandSolder"
 			(at 214.376 148.844 90)
 			(hide yes)
@@
 			)
 		)
-		(property "Footprint" "Resistor_SMD:R_0402_1005Metric"
+		(property "Footprint" "Resistor_SMD:R_0805_2012Metric_Pad1.20x1.40mm_HandSolder"
 			(at 202.946 148.844 90)
 			(hide yes)
@@
 			)
 		)
-		(property "Footprint" "Resistor_SMD:R_0402_1005Metric"
+		(property "Footprint" "Resistor_SMD:R_0805_2012Metric_Pad1.20x1.40mm_HandSolder"
 			(at 252.476 148.844 90)
 			(hide yes)
@@
 			)
 		)
-		(property "Footprint" "Capacitor_SMD:C_0402_1005Metric"
+		(property "Footprint" "Capacitor_SMD:C_0805_2012Metric_Pad1.18x1.45mm_HandSolder"
 			(at 128.27 33.02 0)
 			(hide yes)
@@
 			)
 		)
-		(property "Footprint" "Capacitor_SMD:C_0402_1005Metric"
+		(property "Footprint" "Capacitor_SMD:C_0805_2012Metric_Pad1.18x1.45mm_HandSolder"
 			(at 128.27 26.67 0)
 			(hide yes)
@@
 			)
 		)
-		(property "Footprint" "Capacitor_SMD:C_0402_1005Metric"
+		(property "Footprint" "Capacitor_SMD:C_0805_2012Metric_Pad1.18x1.45mm_HandSolder"
 			(at 118.11 114.3 0)
 			(hide yes)
@@
 			)
 		)
-		(property "Footprint" "Resistor_SMD:R_0402_1005Metric"
+		(property "Footprint" "Resistor_SMD:R_0805_2012Metric_Pad1.20x1.40mm_HandSolder"
 			(at 267.716 148.844 90)
 			(hide yes)
@@
 			)
 		)
-		(property "Footprint" "Resistor_SMD:R_0402_1005Metric"
+		(property "Footprint" "Resistor_SMD:R_0805_2012Metric_Pad1.20x1.40mm_HandSolder"
 			(at 237.236 148.844 90)
 			(hide yes)
@@
 			)
 		)
-		(property "Footprint" "Resistor_SMD:R_0402_1005Metric"
+		(property "Footprint" "Resistor_SMD:R_0805_2012Metric_Pad1.20x1.40mm_HandSolder"
 			(at 244.856 148.844 90)
 			(hide yes)
@@
 			)
 		)
-		(property "Footprint" "Resistor_SMD:R_0402_1005Metric"
+		(property "Footprint" "Resistor_SMD:R_0805_2012Metric_Pad1.20x1.40mm_HandSolder"
 			(at 263.906 148.844 90)
 			(hide yes)
@@
 			)
 		)
-		(property "Footprint" "Resistor_SMD:R_0402_1005Metric"
+		(property "Footprint" "Resistor_SMD:R_0805_2012Metric_Pad1.20x1.40mm_HandSolder"
 			(at 225.806 148.844 90)
 			(hide yes)
