File: ESP32_5V/ESP32_5V.kicad_sch (KiCad schematic)
At the start: 0 parts

Commit message: update
Other:
- sheet Conector_3V3 ports: added D15, D16, D17, D18, D19, D2, D21, D22, D23, D4, D5; removed none
- sheet Conector_5V ports: added D12, D12_5V, D13, D13_5V, D14, D14_5V, D15, D15_5V, D16, D16_5V, D17, D17_5V, D18, D18_5V, D19, D19_5V, D21, D21_5V, D22, D22_5V, D23, D23_5V, D25, D25_5V, D26, D26_5V, D27, D27_5V, D32, D32_5V, D33, D33_5V, D34, D34_5V, D35, D35_5V, D4, D4_5V, D5, D5_5V; removed none
- sheet conector_atornillado ports: added D12_5V, D13_5V, D14_5V, D15_5V, D16_5V, D17_5V, D18_5V, D19_5V, D21_5V, D22_5V, D23_5V, D25_5V, D26_5V, D27_5V, D32_5V, D33_5V, D34_5V, D35_5V, D4_5V, D5_5V; removed none
- note added: "ESP32_5V BOARD"

Commit message: update
Parts:
- added H1, H2, H3, H4: MountingHole_Pad, MountingHole:MountingHole_3.2mm_M3_Pad_Via, symbol Mechanical:MountingHole_Pad
Connections:
- new net GND: H1.1, H2.1, H3.1, H4.1
Other:
- sheet Conector_3V3 ports: added none; removed D23
- sheet Conector_5V ports: added none; removed D23, D23_5V
- sheet ESP32 ports: added none; removed D23
- sheet conector_atornillado ports: added none; removed D23_5V

Commit message: update
Parts:
- added R5: 0, symbol Device:R_US
Connections:
- net GND: now also R5.2; no longer H1.1, H2.1, H3.1, H4.1
- new net: H1.1, R5.1
- no-connect marks 0 -> 3
Changed lines of the file:
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@@
 		(color 0 0 0 0)
 	)
+	(no_connect
+		(at 57.15 177.8)
+	)
+	(no_connect
+		(at 40.64 177.8)
+	)
+	(no_connect
+		(at 49.53 177.8)
+	)
 	(wire
 		(pts
@@
 	(wire
 		(pts
-			(xy 31.75 180.34) (xy 31.75 177.8)
-		)
-		(stroke
-			(width 0)
-			(type default)
-		)
-	)
-	(wire
-		(pts
 			(xy 175.26 82.55) (xy 175.26 64.77)
 		)
@@
 	(wire
 		(pts
-			(xy 40.64 180.34) (xy 40.64 177.8)
-		)
-		(stroke
-			(width 0)
-			(type default)
-		)
-	)
-	(wire
-		(pts
 			(xy 185.42 127.635) (xy 185.42 62.23)
 		)
@@
 	(wire
 		(pts
+			(xy 31.75 187.96) (xy 31.75 186.69)
+		)
+		(stroke
+			(width 0)
+			(type default)
+		)
+	)
+	(wire
+		(pts
 			(xy 176.53 80.01) (xy 176.53 62.23)
 		)
@@
 	(wire
 		(pts
-			(xy 49.53 180.34) (xy 49.53 177.8)
-		)
-		(stroke
-			(width 0)
-			(type default)
-		)
-	)
-	(wire
-		(pts
 			(xy 139.065 97.155) (xy 170.18 97.155)
 		)
@@
 	(wire
 		(pts
-			(xy 57.15 180.34) (xy 57.15 177.8)
-		)
-		(stroke
-			(width 0)
-			(type default)
-		)
-	)
-	(wire
-		(pts
 			(xy 185.42 62.23) (xy 185.42 44.45)
 		)
@@
 		(pts
 			(xy 189.23 54.61) (xy 204.47 54.61)
+		)
+		(stroke
+			(width 0)
+			(type default)
+		)
+	)
+	(wire
+		(pts
+			(xy 31.75 179.07) (xy 31.75 177.8)
 		)
 		(stroke
@@
 	(symbol
 		(lib_id "power:GND")
-		(at 49.53 180.34 0)
-		(unit 1)
-		(exclude_from_sim no)
-		(in_bom yes)
-		(on_board yes)
-		(dnp no)
-		(fields_autoplaced yes)
-		(property "Reference" "#PWR033"
-			(at 49.53 186.69 0)
-			(effects
-				(font
-					(size 1.27 1.27)
-				)
-				(hide yes)
-			)
-		)
-		(property "Value" "GND"
-			(at 49.53 185.42 0)
-			(effects
-				(font
-					(size 1.27 1.27)
-				)
-			)
-		)
-		(property "Footprint" ""
-			(at 49.53 180.34 0)
-			(effects
-				(font
-					(size 1.27 1.27)
-				)
-				(hide yes)
-			)
-		)
-		(property "Datasheet" ""
-			(at 49.53 180.34 0)
-			(effects
-				(font
-					(size 1.27 1.27)
-				)
-				(hide yes)
-			)
-		)
-		(property "Description" "Power symbol creates a global label with name \"GND\" , ground"
-			(at 49.53 180.34 0)
-			(effects
-				(font
-					(size 1.27 1.27)
-				)
-				(hide yes)
-			)
-		)
-		(pin "1"
-		)
-		(instances
-			(project "ESP32_5V"
-				(path "/a7bda8b3-4b40-4c73-a9d2-e587ed8710cd"
-					(reference "#PWR033")
-					(unit 1)
-				)
-			)
-		)
-	)
-	(symbol
-		(lib_id "power:GND")
-		(at 31.75 180.34 0)
+		(at 31.75 187.96 0)
 		(unit 1)
 		(exclude_from_sim no)
@@
 		(fields_autoplaced yes)
 		(property "Reference" "#PWR031"
-			(at 31.75 186.69 0)
+			(at 31.75 194.31 0)
 			(effects
 				(font
@@
 		)
 		(property "Value" "GND"
-			(at 31.75 185.42 0)
+			(at 31.75 193.04 0)
 			(effects
 				(font
@@
 		)
 		(property "Footprint" ""
-			(at 31.75 180.34 0)
+			(at 31.75 187.96 0)
 			(effects
 				(font
@@
 		)
 		(property "Datasheet" ""
-			(at 31.75 180.34 0)
+			(at 31.75 187.96 0)
 			(effects
 				(font
@@
 		)
 		(property "Description" "Power symbol creates a global label with name \"GND\" , ground"
-			(at 31.75 180.34 0)
+			(at 31.75 187.96 0)
 			(effects
 				(font
@@
 	)
 	(symbol
-		(lib_id "power:GND")
-		(at 57.15 180.34 0)
+		(lib_id "Device:R_US")
+		(at 31.75 182.88 0)
 		(unit 1)
 		(exclude_from_sim no)
 		(in_bom yes)
 		(on_board yes)
-		(dnp no)
+		(dnp yes)
 		(fields_autoplaced yes)
-		(property "Reference" "#PWR034"
-			(at 57.15 186.69 0)
-			(effects
-				(font
-					(size 1.27 1.27)
-				)
-				(hide yes)
-			)
-		)
-		(property "Value" "GND"
-			(at 57.15 185.42 0)
-			(effects
-				(font
-					(size 1.27 1.27)
-				)
+		(property "Reference" "R5"
+			(at 34.29 181.6099 0)
+			(effects
+				(font
+					(size 1.27 1.27)
+				)
+				(justify left)
+			)
+		)
+		(property "Value" "0"
+			(at 34.29 184.1499 0)
+			(effects
+				(font
+					(size 1.27 1.27)
+				)
+				(justify left)
 			)
 		)
 		(property "Footprint" ""
-			(at 57.15 180.34 0)
-			(effects
-				(font
-					(size 1.27 1.27)
-				)
-				(hide yes)
-			)
-		)
-		(property "Datasheet" ""
-			(at 57.15 180.34 0)
-			(effects
-				(font
-					(size 1.27 1.27)
-				)
-				(hide yes)
-			)
-		)
-		(property "Description" "Power symbol creates a global label with name \"GND\" , ground"
-			(at 57.15 180.34 0)
-			(effects
-				(font
-					(size 1.27 1.27)
-				)
-				(hide yes)
-			)
+			(at 32.766 183.134 90)
+			(effects
+				(font
+					(size 1.27 1.27)
+				)
+				(hide yes)
+			)
+		)
+		(property "Datasheet" "~"
+			(at 31.75 182.88 0)
+			(effects
+				(font
+					(size 1.27 1.27)
+				)
+				(hide yes)
+			)
+		)
+		(property "Description" "Resistor, US symbol"
+			(at 31.75 182.88 0)
+			(effects
+				(font
+					(size 1.27 1.27)
+				)
+				(hide yes)
+			)
+		)
+		(pin "2"
 		)
 		(pin "1"
 		)
 		(instances
-			(project "ESP32_5V"
+			(project ""
 				(path "/a7bda8b3-4b40-4c73-a9d2-e587ed8710cd"
-					(reference "#PWR034")
+					(reference "R5")
 					(unit 1)
 				)
-			)
-		)
-	)
-	(symbol
-		(lib_id "power:GND")
-		(at 40.64 180.34 0)
-		(unit 1)
-		(exclude_from_sim no)
-		(in_bom yes)
-		(on_board yes)
-		(dnp no)
-		(fields_autoplaced yes)
-		(property "Reference" "#PWR032"
-			(at 40.64 186.69 0)
-			(effects
-				(font
-					(size 1.27 1.27)
-				)
-				(hide yes)
-			)
-		)
-		(property "Value" "GND"
-			(at 40.64 185.42 0)
-			(effects
-				(font
-					(size 1.27 1.27)
-				)
-			)
-		)
-		(property "Footprint" ""
-			(at 40.64 180.34 0)
-			(effects
-				(font
-					(size 1.27 1.27)
-				)
-				(hide yes)
-			)
-		)
-		(property "Datasheet" ""
-			(at 40.64 180.34 0)
-			(effects
-				(font
-					(size 1.27 1.27)
-				)
-				(hide yes)
-			)
-		)
-		(property "Description" "Power symbol creates a global label with name \"GND\" , ground"
-			(at 40.64 180.34 0)
-			(effects
-				(font
-					(size 1.27 1.27)
-				)
-				(hide yes)
-			)
-		)
-		(pin "1"
-		)
-		(instances
-			(project "ESP32_5V"
-				(path "/a7bda8b3-4b40-4c73-a9d2-e587ed8710cd"
-					(reference "#PWR032")
-					(unit 1)
-				)

Commit message: update
Parts:
- R1: renamed from R5; footprint (none) -> Resistor_SMD:R_0402_1005Metric
Changed lines of the file:
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@@
 		(dnp no)
 		(fields_autoplaced yes)
-		(property "Reference" "#PWR031"
+		(property "Reference" "#PWR01"
 			(at 31.75 194.31 0)
 			(effects
@@
 			(project ""
 				(path "/a7bda8b3-4b40-4c73-a9d2-e587ed8710cd"
-					(reference "#PWR031")
+					(reference "#PWR01")
 					(unit 1)
 				)
@@
 		(dnp yes)
 		(fields_autoplaced yes)
-		(property "Reference" "R5"
+		(property "Reference" "R1"
 			(at 34.29 181.6099 0)
 			(effects
@@
 			)
 		)
-		(property "Footprint" ""
+		(property "Footprint" "Resistor_SMD:R_0402_1005Metric"
 			(at 32.766 183.134 90)
 			(effects
@@
 			(project ""
 				(path "/a7bda8b3-4b40-4c73-a9d2-e587ed8710cd"
-					(reference "R5")
-					(unit 1)
-				)
+					(reference "R1")
+					(unit 1)
+				)

Commit message: update
Connections:
- net at H1.1: no longer R1.1
- net at H3.1: now also R1.1
Other:
- moved on the sheet: R1
Changed lines of the file:
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@@
 	)
 	(no_connect
-		(at 49.53 177.8)
+		(at 31.75 177.8)
 	)
 	(wire
@@
 	(wire
 		(pts
-			(xy 31.75 187.96) (xy 31.75 186.69)
-		)
-		(stroke
-			(width 0)
-			(type default)
-		)
-	)
-	(wire
-		(pts
 			(xy 176.53 80.01) (xy 176.53 62.23)
 		)
@@
 	(wire
 		(pts
-			(xy 31.75 179.07) (xy 31.75 177.8)
-		)
-		(stroke
-			(width 0)
-			(type default)
-		)
-	)
-	(wire
-		(pts
 			(xy 180.34 72.39) (xy 204.47 72.39)
 		)
@@
 		(pts
 			(xy 179.07 57.15) (xy 139.7 57.15)
+		)
+		(stroke
+			(width 0)
+			(type default)
+		)
+	)
+	(wire
+		(pts
+			(xy 49.53 179.07) (xy 49.53 177.8)
+		)
+		(stroke
+			(width 0)
+			(type default)
+		)
+	)
+	(wire
+		(pts
+			(xy 49.53 186.69) (xy 49.53 189.23)
 		)
 		(stroke
@@
 	(symbol
 		(lib_id "power:GND")
-		(at 31.75 187.96 0)
+		(at 49.53 189.23 0)
 		(unit 1)
 		(exclude_from_sim no)
@@
 		(fields_autoplaced yes)
 		(property "Reference" "#PWR01"
-			(at 31.75 194.31 0)
+			(at 49.53 195.58 0)
 			(effects
 				(font
@@
 		)
 		(property "Value" "GND"
-			(at 31.75 193.04 0)
+			(at 49.53 194.31 0)
 			(effects
 				(font
@@
 		)
 		(property "Footprint" ""
-			(at 31.75 187.96 0)
+			(at 49.53 189.23 0)
 			(effects
 				(font
@@
 		)
 		(property "Datasheet" ""
-			(at 31.75 187.96 0)
+			(at 49.53 189.23 0)
 			(effects
 				(font
@@
 		)
 		(property "Description" "Power symbol creates a global label with name \"GND\" , ground"
-			(at 31.75 187.96 0)
+			(at 49.53 189.23 0)
 			(effects
 				(font
@@
 		)
 		(instances
-			(project ""
+			(project "ESP32_5V"
 				(path "/a7bda8b3-4b40-4c73-a9d2-e587ed8710cd"
 					(reference "#PWR01")
@@
 	(symbol
 		(lib_id "Device:R_US")
-		(at 31.75 182.88 0)
+		(at 49.53 182.88 0)
 		(unit 1)
 		(exclude_from_sim no)
@@
 		(fields_autoplaced yes)
 		(property "Reference" "R1"
-			(at 34.29 181.6099 0)
+			(at 52.07 181.6099 0)
 			(effects
 				(font
@@
 		)
 		(property "Value" "0"
-			(at 34.29 184.1499 0)
+			(at 52.07 184.1499 0)
 			(effects
 				(font
@@
 		)
 		(property "Footprint" "Resistor_SMD:R_0402_1005Metric"
-			(at 32.766 183.134 90)
+			(at 50.546 183.134 90)
 			(effects
 				(font
@@
 		)
 		(property "Datasheet" "~"
-			(at 31.75 182.88 0)
+			(at 49.53 182.88 0)
 			(effects
 				(font
@@
 		)
 		(property "Description" "Resistor, US symbol"
-			(at 31.75 182.88 0)
+			(at 49.53 182.88 0)
 			(effects
 				(font
@@
 		)
 		(instances
-			(project ""
+			(project "ESP32_5V"
 				(path "/a7bda8b3-4b40-4c73-a9d2-e587ed8710cd"
 					(reference "R1")

Commit message: update
Parts:
- R1: footprint Resistor_SMD:R_0402_1005Metric -> Resistor_SMD:R_0805_2012Metric_Pad1.20x1.40mm_HandSolder
Changed lines of the file:
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@@
 			)
 		)
-		(property "Footprint" "Resistor_SMD:R_0402_1005Metric"
+		(property "Footprint" "Resistor_SMD:R_0805_2012Metric_Pad1.20x1.40mm_HandSolder"
 			(at 50.546 183.134 90)
 			(hide yes)
