File: ESP32_5V/ESP32.kicad_sch (KiCad schematic)
At the start: 3 parts, among them J2 Conn_01x15, J3 Conn_01x15

Commit message: update
Parts:
- removed J2, J3: Conn_01x15, Connector_PinSocket_2.54mm:PinSocket_1x15_P2.54mm_Vertical, symbol Connector_Generic:Conn_01x15
- added J14: ~, ESP32_5V:ESP32_dispositivo, symbol ESP32_5v_library:esp32_board_pins
Connections:
- net D12: now also J14.12
- net D13: now also J14.13
- net D14: now also J14.11
- net D15: now also J14.28
- net D16: now also J14.25
- net D17: now also J14.24
- net D18: now also J14.22
- net D19: now also J14.21
- net D2: now also J14.27
- net D21: now also J14.20
- net D22: now also J14.17
- net D23: now also J14.16
- net D25: now also J14.8
- net D26: now also J14.9
- net D27: now also J14.10
- net D32: now also J14.6
- net D33: now also J14.7
- net D34: now also J14.4
- net D35: now also J14.5
- net D4: now also J14.26
- net D5: now also J14.23
- net GND: now also J14.14, J14.29
- net at JP1.1 (A): now also J14.15
Other:
- moved on the sheet: JP1

Commit message: update
Connections:
- net +3V3: now reaches J14.30
- net D23: no longer names the net of J14.16
Other:
- note added: "ESP32"
- note removed: "(3V3)"
Changed lines of the file:
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@@
 	(generator_version "9.0")
 	(paper "A4")
-	(text "(3V3)"
-		(exclude_from_sim no)
-		(at 163.83 92.71 0)
-		(effects
-			(font
-				(size 1.27 1.27)
-			)
-		)
-	)
 	(text "Solo conectar si el usb c no está conectado"
 		(exclude_from_sim no)
@@
 		)
 	)
+	(text "ESP32"
+		(exclude_from_sim no)
+		(at 144.526 33.528 0)
+		(effects
+			(font
+				(size 3.81 3.81)
+				(thickness 0.762)
+				(bold yes)
+			)
+		)
+	)
 	(no_connect
 		(at 166.37 64.77)
@@
 	)
 	(no_connect
-		(at 158.75 92.71)
+		(at 166.37 57.15)
 	)
 	(no_connect
@@
 	(wire
 		(pts
+			(xy 158.75 92.71) (xy 166.37 92.71)
+		)
+		(stroke
+			(width 0)
+			(type default)
+		)
+	)
+	(wire
+		(pts
 			(xy 158.75 67.31) (xy 166.37 67.31)
 		)
@@
 		(shape bidirectional)
 		(at 166.37 72.39 0)
-		(effects
-			(font
-				(size 1.27 1.27)
-			)
-			(justify left)
-		)
-	)
-	(hierarchical_label "D23"
-		(shape bidirectional)
-		(at 166.37 57.15 0)
 		(effects
 			(font
@@
 					(unit 1)
 				)
+			)
+		)
+	)
+	(symbol
+		(lib_id "power:+3V3")
+		(at 166.37 92.71 270)
+		(unit 1)
+		(exclude_from_sim no)
+		(in_bom yes)
+		(on_board yes)
+		(dnp no)
+		(fields_autoplaced yes)
+		(property "Reference" "#PWR017"
+			(at 162.56 92.71 0)
+			(effects
+				(font
+					(size 1.27 1.27)
+				)
+				(hide yes)
+			)
+		)
+		(property "Value" "+3V3"
+			(at 170.18 92.7099 90)
+			(effects
+				(font
+					(size 1.27 1.27)
+				)
+				(justify left)
+			)
+		)
+		(property "Footprint" ""
+			(at 166.37 92.71 0)
+			(effects
+				(font
+					(size 1.27 1.27)
+				)
+				(hide yes)
+			)
+		)
+		(property "Datasheet" ""
+			(at 166.37 92.71 0)
+			(effects
+				(font
+					(size 1.27 1.27)
+				)
+				(hide yes)
+			)
+		)
+		(property "Description" "Power symbol creates a global label with name \"+3V3\""
+			(at 166.37 92.71 0)
+			(effects
+				(font
+					(size 1.27 1.27)
+				)
+				(hide yes)
+			)
+		)
+		(pin "1"
+		)
+		(instances
+			(project ""
+				(path "/a7bda8b3-4b40-4c73-a9d2-e587ed8710cd/245e545c-c1b3-43e4-a576-56ce0167bab4"
+					(reference "#PWR017")
+					(unit 1)
+				)

Commit message: update
Parts:
- added C12, C13: 10u, Capacitor_SMD:C_0402_1005Metric, symbol Device:C
- added D3: 1N5711UR, Diode_SMD:D_MELF, symbol Diode:1N5711UR
Connections:
- net +3V3: now also C13.1
- net +5V: now also D3.2 (A); no longer JP1.2 (B)
- net GND: now also C12.2, C13.2
- new net: C12.1, D3.1 (K), JP1.2 (B)
Other:
- note added: "*Solo conectar si el usb c no está conectado"
- note removed: "Solo conectar si el usb c no está conectado"

Commit message: update
Parts:
- removed C13: 10u, Capacitor_SMD:C_0402_1005Metric, symbol Device:C
- removed D3: 1N5711UR, Diode_SMD:D_MELF, symbol Diode:1N5711UR
- added D4: 1N5819WS, Diode_SMD:D_SOD-323, symbol Diode:1N5819WS
- renumbered C12 to C30
Connections:
- net +5V: now also D4.2 (A)
- net at C30.1, JP1.2 (B): now also D4.1 (K)
- net +3V3: no longer names the net of J14.30
- no-connect marks 6 -> 7
Other:
- note added: "*Alimentación independiente Solo conectar si el usb c no está conectado"
- note removed: "*Solo conectar si el usb c no está conectado"

Commit message: update
Parts:
- removed D4: 1N5819WS, Diode_SMD:D_SOD-323, symbol Diode:1N5819WS
- C30: footprint Capacitor_SMD:C_0402_1005Metric -> Capacitor_SMD:C_1206_3216Metric
Connections:
- net +5V: now also C30.1, JP1.2 (B)
Changed lines of the file:
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@@
 	(wire
 		(pts
-			(xy 105.41 92.71) (xy 110.49 92.71)
+			(xy 116.84 92.71) (xy 121.92 92.71)
 		)
 		(stroke
@@
 	(wire
 		(pts
-			(xy 105.41 90.17) (xy 105.41 92.71)
+			(xy 116.84 90.17) (xy 116.84 92.71)
 		)
 		(stroke
@@
 		(pts
 			(xy 135.89 74.93) (xy 128.27 74.93)
-		)
-		(stroke
-			(width 0)
-			(type default)
-		)
-	)
-	(wire
-		(pts
-			(xy 118.11 92.71) (xy 121.92 92.71)
 		)
 		(stroke
@@
 			)
 		)
-		(property "Footprint" "Capacitor_SMD:C_0402_1005Metric"
+		(property "Footprint" "Capacitor_SMD:C_1206_3216Metric"
 			(at 122.8852 109.22 0)
 			(effects
@@
 	(symbol
 		(lib_id "power:+5V")
-		(at 105.41 90.17 0)
+		(at 116.84 90.17 0)
 		(unit 1)
 		(exclude_from_sim no)
@@
 		(dnp no)
 		(property "Reference" "#PWR050"
-			(at 105.41 93.98 0)
+			(at 116.84 93.98 0)
 			(effects
 				(font
@@
 		)
 		(property "Value" "+5V"
-			(at 101.854 86.106 0)
+			(at 113.284 86.106 0)
 			(effects
 				(font
@@
 		)
 		(property "Footprint" ""
-			(at 105.41 90.17 0)
+			(at 116.84 90.17 0)
 			(effects
 				(font
@@
 		)
 		(property "Datasheet" ""
-			(at 105.41 90.17 0)
+			(at 116.84 90.17 0)
 			(effects
 				(font
@@
 		)
 		(property "Description" "Power symbol creates a global label with name \"+5V\""
-			(at 105.41 90.17 0)
+			(at 116.84 90.17 0)
 			(effects
 				(font
@@
 					(unit 1)
 				)
-			)
-		)
-	)
-	(symbol
-		(lib_id "Diode:1N5819WS")
-		(at 114.3 92.71 180)
-		(unit 1)
-		(exclude_from_sim no)
-		(in_bom yes)
-		(on_board yes)
-		(dnp no)
-		(property "Reference" "D4"
-			(at 114.6175 99.06 0)
-			(effects
-				(font
-					(size 1.27 1.27)
-				)
-			)
-		)
-		(property "Value" "1N5819WS"
-			(at 114.6175 96.52 0)
-			(effects
-				(font
-					(size 1.27 1.27)
-				)
-			)
-		)
-		(property "Footprint" "Diode_SMD:D_SOD-323"
-			(at 114.3 88.265 0)
-			(effects
-				(font
-					(size 1.27 1.27)
-				)
-				(hide yes)
-			)
-		)
-		(property "Datasheet" "https://datasheet.lcsc.com/lcsc/2204281430_Guangdong-Hottech-1N5819WS_C191023.pdf"
-			(at 114.3 92.71 0)
-			(effects
-				(font
-					(size 1.27 1.27)
-				)
-				(hide yes)
-			)
-		)
-		(property "Description" "40V 600mV@1A 1A SOD-323 Schottky Barrier Diodes, SOD-323"
-			(at 114.3 92.71 0)
-			(effects
-				(font
-					(size 1.27 1.27)
-				)
-				(hide yes)
-			)
-		)
-		(pin "2"
-		)
-		(pin "1"
-		)
-		(instances
-			(project ""
-				(path "/a7bda8b3-4b40-4c73-a9d2-e587ed8710cd/245e545c-c1b3-43e4-a576-56ce0167bab4"
-					(reference "D4")
-					(unit 1)
-				)

Commit message: update
Parts:
- removed JP1: Jumper_2_Open, Connector_PinHeader_2.54mm:PinHeader_1x02_P2.54mm_Vertical, symbol Jumper:Jumper_2_Open
- added D4: 1N5712UR, Diode_SMD:D_MELF, symbol Diode:1N5712UR
Connections:
- net +5V: now also D4.2 (A); no longer C30.1
- net at J14.15: now also C30.1, D4.1 (K)
Other:
- note removed: "*Alimentación independiente Solo conectar si el usb c no está conectado"
- moved on the sheet: C30
Changed lines of the file:
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@@
 	(generator_version "9.0")
 	(paper "A4")
-	(text "*Alimentación independiente\nSolo conectar si el usb c \nno está conectado"
-		(exclude_from_sim no)
-		(at 143.51 102.362 0)
-		(effects
-			(font
-				(size 1.27 1.27)
-				(thickness 0.254)
-				(bold yes)
-				(italic yes)
-			)
-		)
-	)
 	(text "ESP32"
 		(exclude_from_sim no)
@@
 	)
 	(junction
-		(at 121.92 92.71)
+		(at 133.35 92.71)
 		(diameter 0)
 		(color 0 0 0 0)
@@
 	(wire
 		(pts
-			(xy 116.84 92.71) (xy 121.92 92.71)
-		)
-		(stroke
-			(width 0)
-			(type default)
-		)
-	)
-	(wire
-		(pts
 			(xy 135.89 64.77) (xy 128.27 64.77)
 		)
@@
 	(wire
 		(pts
-			(xy 121.92 92.71) (xy 124.46 92.71)
-		)
-		(stroke
-			(width 0)
-			(type default)
-		)
-	)
-	(wire
-		(pts
 			(xy 135.89 59.69) (xy 128.27 59.69)
 		)
@@
 	(wire
 		(pts
+			(xy 133.35 92.71) (xy 135.89 92.71)
+		)
+		(stroke
+			(width 0)
+			(type default)
+		)
+	)
+	(wire
+		(pts
 			(xy 158.75 72.39) (xy 166.37 72.39)
 		)
@@
 	(wire
 		(pts
-			(xy 116.84 90.17) (xy 116.84 92.71)
-		)
-		(stroke
-			(width 0)
-			(type default)
-		)
-	)
-	(wire
-		(pts
 			(xy 135.89 85.09) (xy 128.27 85.09)
 		)
@@
 	(wire
 		(pts
-			(xy 121.92 109.22) (xy 121.92 110.49)
+			(xy 133.35 102.87) (xy 133.35 104.14)
 		)
 		(stroke
@@
 	(wire
 		(pts
-			(xy 121.92 101.6) (xy 121.92 92.71)
+			(xy 133.35 95.25) (xy 133.35 92.71)
 		)
 		(stroke
@@
 	(wire
 		(pts
-			(xy 134.62 92.71) (xy 135.89 92.71)
+			(xy 121.92 92.71) (xy 123.19 92.71)
 		)
 		(stroke
@@
 		(pts
 			(xy 158.75 57.15) (xy 166.37 57.15)
+		)
+		(stroke
+			(width 0)
+			(type default)
+		)
+	)
+	(wire
+		(pts
+			(xy 130.81 92.71) (xy 133.35 92.71)
 		)
 		(stroke
@@
 	(symbol
 		(lib_id "Device:C")
-		(at 121.92 105.41 0)
+		(at 133.35 99.06 0)
 		(unit 1)
 		(exclude_from_sim no)
@@
 		(dnp no)
 		(property "Reference" "C30"
-			(at 125.222 104.14 0)
+			(at 136.652 97.79 0)
 			(effects
 				(font
@@
 		)
 		(property "Value" "10u"
-			(at 125.222 106.934 0)
+			(at 136.652 100.584 0)
 			(effects
 				(font
@@
 		)
 		(property "Footprint" "Capacitor_SMD:C_1206_3216Metric"
-			(at 122.8852 109.22 0)
+			(at 134.3152 102.87 0)
 			(effects
 				(font
@@
 		)
 		(property "Datasheet" "~"
-			(at 121.92 105.41 0)
+			(at 133.35 99.06 0)
 			(effects
 				(font
@@
 		)
 		(property "Description" "Unpolarized capacitor"
-			(at 121.92 105.41 0)
+			(at 133.35 99.06 0)
 			(effects
 				(font
@@
 		)
 		(property "Sim.Device" ""
-			(at 121.92 105.41 0)
+			(at 133.35 99.06 0)
 			(effects
 				(font
@@
 		)
 		(property "Sim.Pins" ""
-			(at 121.92 105.41 0)
+			(at 133.35 99.06 0)
 			(effects
 				(font
@@
 		)
 		(property "Sim.Type" ""
-			(at 121.92 105.41 0)
+			(at 133.35 99.06 0)
 			(effects
 				(font
@@
 				(path "/a7bda8b3-4b40-4c73-a9d2-e587ed8710cd/245e545c-c1b3-43e4-a576-56ce0167bab4"
 					(reference "C30")
-					(unit 1)
-				)
-			)
-		)
-	)
-	(symbol
-		(lib_id "Jumper:Jumper_2_Open")
-		(at 129.54 92.71 180)
-		(unit 1)
-		(exclude_from_sim no)
-		(in_bom yes)
-		(on_board yes)
-		(dnp no)
-		(property "Reference" "JP1"
-			(at 124.968 95.25 0)
-			(effects
-				(font
-					(size 1.27 1.27)
-				)
-			)
-		)
-		(property "Value" "Jumper_2_Open"
-			(at 136.652 96.266 0)
-			(effects
-				(font
-					(size 1.27 1.27)
-				)
-			)
-		)
-		(property "Footprint" "Connector_PinHeader_2.54mm:PinHeader_1x02_P2.54mm_Vertical"
-			(at 129.54 92.71 0)
-			(effects
-				(font
-					(size 1.27 1.27)
-				)
-				(hide yes)
-			)
-		)
-		(property "Datasheet" "~"
-			(at 129.54 92.71 0)
-			(effects
-				(font
-					(size 1.27 1.27)
-				)
-				(hide yes)
-			)
-		)
-		(property "Description" "Jumper, 2-pole, open"
-			(at 129.54 92.71 0)
-			(effects
-				(font
-					(size 1.27 1.27)
-				)
-				(hide yes)
-			)
-		)
-		(pin "1"
-		)
-		(pin "2"
-		)
-		(instances
-			(project ""
-				(path "/a7bda8b3-4b40-4c73-a9d2-e587ed8710cd/245e545c-c1b3-43e4-a576-56ce0167bab4"
-					(reference "JP1")
-					(unit 1)
-				)
-			)
-			(project "ESP32"
-				(path "/ce980e7b-dd96-46ab-b712-358a93796c11"
-					(reference "JP?")
 					(unit 1)
 				)
@@
 	)
 	(symbol
+		(lib_id "Diode:1N5712UR")
+		(at 127 92.71 180)
+		(unit 1)
+		(exclude_from_sim no)
+		(in_bom yes)
+		(on_board yes)
+		(dnp no)
+		(property "Reference" "D4"
+			(at 127 98.298 0)
+			(effects
+				(font
+					(size 1.27 1.27)
+				)
+			)
+		)
+		(property "Value" "1N5712UR"
+			(at 126.746 95.504 0)
+			(effects
+				(font
+					(size 1.27 1.27)
+				)
+			)
+		)
+		(property "Footprint" "Diode_SMD:D_MELF"
+			(at 127 88.265 0)
+			(effects
+				(font
+					(size 1.27 1.27)
+				)
+				(hide yes)
+			)
+		)
+		(property "Datasheet" "https://www.microsemi.com/document-portal/doc_download/131890-lds-0040-1-datasheet"
+			(at 127 92.71 0)
+			(effects
+				(font
+					(size 1.27 1.27)
+				)
+				(hide yes)
+			)
+		)
+		(property "Description" "20V 75mA Schottky diode, MELF(DO-213AA)"
+			(at 127 92.71 0)
+			(effects
+				(font
+					(size 1.27 1.27)
+				)
+				(hide yes)
+			)
+		)
+		(pin "2"
+		)
+		(pin "1"
+		)
+		(instances
+			(project ""
+				(path "/a7bda8b3-4b40-4c73-a9d2-e587ed8710cd/245e545c-c1b3-43e4-a576-56ce0167bab4"
+					(reference "D4")
+					(unit 1)
+				)
+			)
+		)
+	)
+	(symbol
 		(lib_id "power:GND")
 		(at 166.37 90.17 90)
@@
 	(symbol
 		(lib_id "power:GND")
-		(at 121.92 110.49 0)
+		(at 133.35 104.14 0)
 		(unit 1)
 		(exclude_from_sim no)
@@
 		(fields_autoplaced yes)
 		(property "Reference" "#PWR051"
-			(at 121.92 116.84 0)
+			(at 133.35 110.49 0)
 			(effects
 				(font
@@
 		)
 		(property "Value" "GND"
-			(at 124.46 111.7599 0)
+			(at 135.89 105.4099 0)
 			(effects
 				(font
@@
 		)
 		(property "Footprint" ""
-			(at 121.92 110.49 0)
+			(at 133.35 104.14 0)
 			(effects
 				(font
@@
 		)
 		(property "Datasheet" ""
-			(at 121.92 110.49 0)
+			(at 133.35 104.14 0)
 			(effects
 				(font
@@
 		)
 		(property "Description" "Power symbol creates a global label with name \"GND\" , ground"
-			(at 121.92 110.49 0)
+			(at 133.35 104.14 0)
 			(effects
 				(font
@@
 	(symbol
 		(lib_id "power:+5V")
-		(at 116.84 90.17 0)
+		(at 121.92 92.71 90)
 		(unit 1)
 		(exclude_from_sim no)
@@
 		(dnp no)
 		(property "Reference" "#PWR050"
-			(at 116.84 93.98 0)
+			(at 125.73 92.71 0)
 			(effects
 				(font
@@
 		)
 		(property "Value" "+5V"
-			(at 113.284 86.106 0)
+			(at 118.11 92.202 90)
 			(effects
 				(font
@@
 		)
 		(property "Footprint" ""
-			(at 116.84 90.17 0)
+			(at 121.92 92.71 0)
 			(effects
 				(font
@@
 		)
 		(property "Datasheet" ""
-			(at 116.84 90.17 0)
+			(at 121.92 92.71 0)
 			(effects
 				(font
@@
 		)
 		(property "Description" "Power symbol creates a global label with name \"+5V\""
-			(at 116.84 90.17 0)
-			(effects
-				(font
+			(at 121.92 92.71 0)
+			(effects
+				(font

Commit message: update
Parts:
- J14: value ~ -> (none)

Commit message: update
Parts:
- removed D4: 1N5712UR, Diode_SMD:D_MELF, symbol Diode:1N5712UR
- added D5: 1N5819WS, Diode_SMD:D_SOD-323, symbol Diode:1N5819WS
Connections:
- net +5V: now also D5.2 (A)
- net at C30.1, J14.15: now also D5.1 (K)
Changed lines of the file:
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@@
-	)
-	(symbol
-		(lib_id "Diode:1N5712UR")
-		(at 127 92.71 180)
-		(unit 1)
-		(body_style 1)
-		(exclude_from_sim no)
-		(in_bom yes)
-		(on_board yes)
-		(in_pos_files yes)
-		(dnp no)
-		(property "Reference" "D4"
-			(at 127 98.298 0)
-			(show_name no)
-			(do_not_autoplace no)
-			(effects
-				(font
-					(size 1.27 1.27)
-				)
-			)
-		)
-		(property "Value" "1N5712UR"
-			(at 126.746 95.504 0)
-			(show_name no)
-			(do_not_autoplace no)
-			(effects
-				(font
-					(size 1.27 1.27)
-				)
-			)
-		)
-		(property "Footprint" "Diode_SMD:D_MELF"
-			(at 127 88.265 0)
-			(hide yes)
-			(show_name no)
-			(do_not_autoplace no)
-			(effects
-				(font
-					(size 1.27 1.27)
-				)
-			)
-		)
-		(property "Datasheet" "https://www.microsemi.com/document-portal/doc_download/131890-lds-0040-1-datasheet"
-			(at 127 92.71 0)
-			(hide yes)
-			(show_name no)
-			(do_not_autoplace no)
-			(effects
-				(font
-					(size 1.27 1.27)
-				)
-			)
-		)
-		(property "Description" "20V 75mA Schottky diode, MELF(DO-213AA)"
-			(at 127 92.71 0)
-			(hide yes)
-			(show_name no)
-			(do_not_autoplace no)
-			(effects
-				(font
-					(size 1.27 1.27)
-				)
-			)
-		)
-		(pin "2"
-		)
-		(pin "1"
-		)
-		(instances
-			(project "ESP32_5V"
-				(path "/a7bda8b3-4b40-4c73-a9d2-e587ed8710cd/245e545c-c1b3-43e4-a576-56ce0167bab4"
-					(reference "D4")
-					(unit 1)
-				)
-			)
-		)
 	)
 	(symbol
@@
 					(unit 1)
 				)
+			)
+		)
+	)
+	(symbol
+		(lib_id "Diode:1N5819WS")
+		(at 127 92.71 180)
+		(unit 1)
+		(body_style 1)
+		(exclude_from_sim no)
+		(in_bom yes)
+		(on_board yes)
+		(in_pos_files yes)
+		(dnp no)
+		(property "Reference" "D5"
+			(at 131.318 94.742 0)
+			(show_name no)
+			(do_not_autoplace no)
+			(effects
+				(font
+					(size 1.27 1.27)
+				)
+			)
+		)
+		(property "Value" "1N5819WS"
+			(at 124.206 96.52 0)
+			(show_name no)
+			(do_not_autoplace no)
+			(effects
+				(font
+					(size 1.27 1.27)
+				)
+			)
+		)
+		(property "Footprint" "Diode_SMD:D_SOD-323"
+			(at 127 88.265 0)
+			(hide yes)
+			(show_name no)
+			(do_not_autoplace no)
+			(effects
+				(font
+					(size 1.27 1.27)
+				)
+			)
+		)
+		(property "Datasheet" "https://datasheet.lcsc.com/lcsc/2204281430_Guangdong-Hottech-1N5819WS_C191023.pdf"
+			(at 127 92.71 0)
+			(hide yes)
+			(show_name no)
+			(do_not_autoplace no)
+			(effects
+				(font
+					(size 1.27 1.27)
+				)
+			)
+		)
+		(property "Description" "40V 600mV@1A 1A SOD-323 Schottky Barrier Diodes, SOD-323"
+			(at 127 92.71 0)
+			(hide yes)
+			(show_name no)
+			(do_not_autoplace no)
+			(effects
+				(font
+					(size 1.27 1.27)
+				)
+			)
+		)
+		(pin "1"
+		)
+		(pin "2"
+		)
+		(instances
+			(project "ESP32_5V"
+				(path "/a7bda8b3-4b40-4c73-a9d2-e587ed8710cd/245e545c-c1b3-43e4-a576-56ce0167bab4"
+					(reference "D5")
+					(unit 1)
+				)
